Commit message: update the wheel urdf xacro with the updated info from solidworks

File: omni_base_description/urdf/wheels/wheel.urdf.xacro (robot description, xacro)
@@ -11,25 +11,63 @@
   <xacro:include filename="$(find omni_base_description)/urdf/wheels/wheel.transmission.xacro"/>
   <xacro:include filename="$(find omni_base_description)/urdf/wheels/wheel.gazebo.xacro"/>
-  <xacro:macro name="wheel" params="side reflect radius width torque velocity pair_separation separation parent">
+  <!-- frontal_reflect: front: +1 and rear: -1 -->
+  <!-- sagital_reflect: right: +1 and left: -1 -->
+  <xacro:macro name="wheel" params="side parent sagital_reflect frontal_reflect radius width torque velocity sagital_separation frontal_separation">
+    <link name="suspension_${side}_link">
+      <inertial>
+        <origin xyz="-0.058182 ${frontal_reflect * sagital_reflect * -0.0043908} -0.0057695" rpy="0 0 0" />
+        <mass value="1.2879" />
+        <inertia ixx="0.0015947" ixy="${frontal_reflect * sagital_reflect * -0.00013183}" ixz="1.7315E-05"
+          iyy="0.00060158" iyz="${frontal_reflect * sagital_reflect * -6.0731E-05}" izz="0.0015861" />
+      </inertial>
+      <visual>
+        <origin xyz="0 0 0" rpy="0 0 0" />
+        <geometry>
+          <xacro:if value="${frontal_reflect == 1}">
+            <mesh filename="package://omni_base_description/meshes/wheels/suspension_front_link.stl" scale="1 ${sagital_reflect} 1"/>
+          </xacro:if>
+          <xacro:unless value="${frontal_reflect == 1}">
+            <mesh filename="package://omni_base_description/meshes/wheels/suspension_rear_link.stl" scale="1 ${sagital_reflect} 1"/>
+          </xacro:unless>
+        </geometry>
+        <material name="">
+          <color rgba="0.79216 0.81961 0.93333 1" />
+        </material>
+      </visual>
+      <collision>
+        <origin xyz="0 0 0" rpy="0 0 0" />
+        <geometry>
+          <xacro:if value="${frontal_reflect == 1}">
+            <mesh filename="package://omni_base_description/meshes/wheels/suspension_front_link.stl" scale="1 ${sagital_reflect} 1"/>
+          </xacro:if>
+          <xacro:unless value="${frontal_reflect == 1}">
+            <mesh filename="package://omni_base_description/meshes/wheels/suspension_rear_link.stl" scale="1 ${sagital_reflect} 1"/>
+          </xacro:unless>
+        </geometry>
+      </collision>
+      <kinematic>0</kinematic>
+      <gravity>1</gravity>
+    </link>
+    <joint name="suspension_${side}_joint" type="prismatic">
+      <origin xyz="${frontal_reflect * frontal_separation / 2.0} ${sagital_reflect * -1.0 * suspension_sagital_separation / 2.0} 0" rpy="0 0 ${sagital_reflect * -90.0 * deg_to_rad}" />
+      <parent link="${parent}" />
+      <child link="suspension_${side}_link" />
+      <axis xyz="0 0 1" />
+      <calibration rising="0.0" />
+      <dynamics damping="100"/>
+      <limit lower="-0.01" upper="0.01" effort="100" velocity="1.0" />
+    </joint>
     <link name="wheel_${side}_link">
       <inertial>
-        <origin xyz="0 0 ${-0.00207 * reflect}" rpy="0 0 0"/>
-        <mass value="1.82362"/>
-        <inertia ixx="0.00499743171" ixy="${ 0.00000004464 * reflect}" ixz="-0.00000002245"
-          iyy="0.00499741733" iyz="${-0.00000000164 * reflect}"
-          izz="0.00839239692"/>
+        <origin xyz="${frontal_reflect * 5.4922E-09} ${frontal_reflect * sagital_reflect * 6.9775E-05} ${sagital_reflect * 0.011144}" rpy="0 0 0" />
+        <mass value="0.70767" />
+        <inertia ixx="0.00035492" ixy="${frontal_reflect * 7.5685E-13}" ixz="3.8795E-11"
+          iyy="0.00035529" iyz="${frontal_reflect * -2.0284E-07}" izz="0.00040131" />
       </inertial>
       <visual>
-        <origin xyz="0 0 0" rpy="${-90.0 * deg_to_rad} 0 0"/>
-        <xacro:if value="${reflect == '1'}">
-          <geometry>
-            <mesh filename="package://omni_base_description/meshes/wheels/wheel_1.stl" scale="0.8 0.8 0.8"/>
-          </geometry>
-        </xacro:if>
-        <xacro:unless value="${reflect == '1'}">
-          <geometry>
-            <mesh filename="package://omni_base_description/meshes/wheels/wheel_2.stl" scale="0.8 0.8 0.8"/>
-          </geometry>
-		    </xacro:unless>
+        <origin xyz="0 0 0" rpy="0 0 0" />
+        <geometry>
+          <mesh filename="package://omni_base_description/meshes/wheels/wheel_link.stl" scale="1 1 ${sagital_reflect}"/>
+        </geometry>
         <material name="DarkGrey"/>
       </visual>
@@ -37,37 +75,13 @@
         <origin xyz="0 0 0" rpy="0 0 0" />
         <geometry>
-					<cylinder radius="${radius}" length="${width}"/>
+          <cylinder radius="${radius}" length="${width}"/>
         </geometry>
       </collision>
     </link>
-    <link name="suspension_${side}_link">
-      <inertial>
-        <origin xyz="0 0 -0.02" rpy="0 0 0"/>
-        <mass value="10"/>
-        <inertia ixx="1.0" ixy="0" ixz="0"
-                  iyy="1.0" iyz="0"
-                  izz="1.0"/>
-      </inertial>
-      <kinematic>0</kinematic>
-      <gravity>1</gravity>
-    </link>
-    <joint name="suspension_${side}_joint" type="prismatic">
-      <origin xyz="${pair_separation / 2} 0 0" rpy="0 0 0"/>
-      <axis xyz="0 0 1"/>
-      <limit effort="100.0" lower="-0.005" upper="0.005" velocity="1.0"/>
-      <child link="suspension_${side}_link"/>
-      <parent link="${parent}_link"/>
-      <calibration rising="0.0" />
-      <dynamics damping="100"/>
-      <safety_controller k_position="0"
-        k_velocity="10"
-        soft_lower_limit="-0.005"
-        soft_upper_limit="0.005" />
-    </joint>
     <joint name="wheel_${side}_joint" type="continuous">
-      <parent link="suspension_${side}_link"/>
-      <child link="wheel_${side}_link"/>
-      <origin xyz="0 ${-separation / 2 * reflect} 0" rpy="${-90.0 * deg_to_rad} 0 0"/>
-      <axis xyz="0 0 1"/>
+      <origin xyz="0.050675 0 0" rpy="${-90.0 * deg_to_rad} 0 ${sagital_reflect * 90.0 * deg_to_rad}" />
+      <parent link="suspension_${side}_link" />
+      <child link="wheel_${side}_link" />
+      <axis xyz="0 0 1" />
       <limit effort="${torque}" velocity="${velocity / radius}"/>
     </joint>

Commit message: Change suspension_side_joints to fixed joint because it was causing issue in the odometry

File: omni_base_description/urdf/wheels/wheel.urdf.xacro (robot description, xacro)
@@ -49,12 +49,10 @@
       <gravity>1</gravity>
     </link>
-    <joint name="suspension_${side}_joint" type="prismatic">
+    <!-- Changed joint type to fixed joint. It is observed that the robot is loosing contact points due to some issues with the Gazebo Physics Engine. This makes the robot drift in localization when static due to added noise -->
+    <joint name="suspension_${side}_joint" type="fixed">
       <origin xyz="${frontal_reflect * frontal_separation / 2.0} ${sagital_reflect * -1.0 * suspension_sagital_separation / 2.0} 0" rpy="0 0 ${sagital_reflect * -90.0 * deg_to_rad}" />
       <parent link="${parent}" />
       <child link="suspension_${side}_link" />
       <axis xyz="0 0 1" />
-      <calibration rising="0.0" />
-      <dynamics damping="100"/>
-      <limit lower="-0.01" upper="0.01" effort="100" velocity="1.0" />
     </joint>
     <link name="wheel_${side}_link">
