Commit message: omnibase description to ROS 2: + xacro + ros2_control + launch.py

File: omni_base_description/gazebo/gazebo.urdf.xacro (robot description, xacro)
@@ -1,24 +1,29 @@
 <?xml version="1.0"?>
 <!--
-  Copyright (c) 2011, PAL Robotics, S.L.
+  Copyright (c) 2023, PAL Robotics, S.L.
   All rights reserved.
-  This work is licensed under the Creative Commons Attribution-NonCommercial-NoDerivs 3.0 Unported License.
-  To view a copy of this license, visit http://creativecommons.org/licenses/by-nc-nd/3.0/ or send a letter to
-  Creative Commons, 444 Castro Street, Suite 900, Mountain View, California, 94041, USA.
+  Licensed under the Apache License, Version 2.0 (the "License");
+  you may not use this file except in compliance with the License.
+  You may obtain a copy of the License at
+      http://www.apache.org/licenses/LICENSE-2.0
+  Unless required by applicable law or agreed to in writing, software
+  distributed under the License is distributed on an "AS IS" BASIS,
+  WITHOUT WARRANTIES OR CONDITIONS OF ANY KIND, either express or implied.
+  See the License for the specific language governing permissions and
+  limitations under the License.
 -->
 <robot name="omni_base" xmlns:xacro="http://ros.org/wiki/xacro">
   <gazebo>
-    <plugin filename="libgazebo_ros_control.so" name="gazebo_ros_control">
-      <ns></ns>
-      <robotSimType>pal_hardware_gazebo/PalHardwareGazebo</robotSimType>
+    <plugin filename="libgazebo_ros2_control.so" name="gazebo_ros2_control">
+      <robot_sim_type>gazebo_ros2_control/GazeboSystem</robot_sim_type>
+      <control_period>0.001</control_period>
       <xacro:if value="${is_multiple}">
-          <robotNamespace>/${nsp}</robotNamespace>
+        <!-- Do something about multirobot -->
       </xacro:if>
       <xacro:unless value="${is_multiple}">
-          <robotNamespace></robotNamespace>
+        <!-- Do something about multirobot -->
       </xacro:unless>
-      <controlPeriod>0.001</controlPeriod>
     </plugin>
-    <plugin filename="libgazebo_ros_force_based_move.so" name="gazebo_force_based_move" >
+    <!--<plugin filename="libgazebo_ros_force_based_move.so" name="gazebo_force_based_move" >
       <commandTopic>mobile_base_controller/cmd_vel</commandTopic>
       <odometryTopic>mobile_base_controller/odom</odometryTopic>
@@ -27,5 +32,5 @@
       <robotBaseFrame>base_footprint</robotBaseFrame>
       <publishOdometryTf>true</publishOdometryTf>
-    </plugin>
+    </plugin>-->
   </gazebo>
   <gazebo reference="base_imu_link">

File: omni_base_description/robots/omni_base.urdf.xacro (robot description, xacro)
@@ -1,11 +1,17 @@
 <?xml version="1.0"?>
 <!--
-  Copyright (c) 2021, PAL Robotics, S.L.
-  All rights reserved.
-  This work is licensed under the Creative Commons Attribution-NonCommercial-NoDerivs 3.0 Unported License.
-  To view a copy of this license, visit http://creativecommons.org/licenses/by-nc-nd/3.0/ or send a letter to
-  Creative Commons, 444 Castro Street, Suite 900, Mountain View, California, 94041, USA.
--->
+  Copyright (c) 2023 PAL Robotics S.L. All rights reserved.
+  Licensed under the Apache License, Version 2.0 (the "License");
+  you may not use this file except in compliance with the License.
+  You may obtain a copy of the License at
+      http://www.apache.org/licenses/LICENSE-2.0
+  Unless required by applicable law or agreed to in writing, software
+  distributed under the License is distributed on an "AS IS" BASIS,
+  WITHOUT WARRANTIES OR CONDITIONS OF ANY KIND, either express or implied.
+  See the License for the specific language governing permissions and
+  limitations under the License.
+ -->
 <robot  xmlns:xacro="http://ros.org/wiki/xacro" name="omni_base" >
+  <xacro:arg name="use_sim" default="true"/>
   <xacro:arg name="front_laser_model" default="sick-571"/> <!-- false, hokuyo, sick-551, sick-561, sick-571-->
   <xacro:arg name="rear_laser_model" default="sick-571"/> <!-- false, hokuyo, sick-551, sick-561, sick-571-->
@@ -27,4 +33,7 @@
   <!-- Generic simulator_gazebo plugins -->
   <xacro:include filename="$(find omni_base_description)/gazebo/gazebo.urdf.xacro" />
+  <!-- ros2_control -->
+  <xacro:include filename="$(find omni_base_description)/ros2_control/ros2_control.urdf.xacro" />
+  <xacro:omni_base_ros2_control use_sim="$(arg use_sim)" />
   <!-- Materials for visualization -->
   <xacro:include filename="$(find omni_base_description)/urdf/materials.urdf.xacro" />

File: omni_base_description/urdf/base/antenna.urdf.xacro (robot description, xacro)
@@ -1,5 +1,5 @@
 <?xml version="1.0"?>
 <!--
-  Copyright (c) 2021 PAL Robotics S.L. All rights reserved.
+  Copyright (c) 2023 PAL Robotics S.L. All rights reserved.
   Licensed under the Apache License, Version 2.0 (the "License");
   you may not use this file except in compliance with the License.
@@ -11,5 +11,5 @@
   See the License for the specific language governing permissions and
   limitations under the License.
--->
+ -->
 <robot xmlns:xacro="http://ros.org/wiki/xacro">
   <xacro:macro name="antenna" params="name parent *origin reflect:=1">

File: omni_base_description/urdf/wheels/wheel.gazebo.xacro (robot description, xacro)
@@ -1,10 +1,14 @@
 <!--
- Copyright 2021 PAL Robotics SL.
- All Rights Reserved
- Unauthorized copying of this file, via any medium is strictly prohibited,
- unless it was supplied under the terms of a license agreement or
- nondisclosure agreement with PAL Robotics SL. In this case it may not be
- copied or disclosed except in accordance with the terms of that agreement.
--->
+  Copyright (c) 2023 PAL Robotics S.L. All rights reserved.
+  Licensed under the Apache License, Version 2.0 (the "License");
+  you may not use this file except in compliance with the License.
+  You may obtain a copy of the License at
+      http://www.apache.org/licenses/LICENSE-2.0
+  Unless required by applicable law or agreed to in writing, software
+  distributed under the License is distributed on an "AS IS" BASIS,
+  WITHOUT WARRANTIES OR CONDITIONS OF ANY KIND, either express or implied.
+  See the License for the specific language governing permissions and
+  limitations under the License.
+ -->
 <robot xmlns:xacro="http://ros.org/wiki/xacro">
   <xacro:macro name="wheel_gazebo" params="side">
@@ -13,12 +17,23 @@
       <kp>1000000.0</kp>
       <kd>1000.0</kd>
-      <mu1>0.0</mu1>
-      <mu2>0.0</mu2>
-      <fdir1>1 0 0</fdir1>
-      <maxVel>1.0</maxVel>
-      <minDepth>0.00</minDepth>
+      <friction>
+        <ode>
+          <mu>0.0</mu>
+          <mu2>0.0</mu2>
+        </ode>
+      </friction>
+      <!--<fdir1>1 0 0</fdir1>-->
+      <max_vel>1.0</max_vel>
+      <min_depth>0.0</min_depth>
       <implicitSpringDamper>1</implicitSpringDamper>
       <material>Gazebo/DarkGrey</material>
     </gazebo>
+    <gazebo reference="wheel_{side}_joint">
+      <physics>
+        <ode>
+          <implicit_spring_damper>1</implicit_spring_damper>
+        </ode>
+      </physics>
+    </gazebo>
   </xacro:macro>
 </robot>

File: omni_base_description/urdf/wheels/wheel.urdf.xacro (robot description, xacro)
@@ -1,13 +1,17 @@
 <?xml version="1.0"?>
 <!--
-Copyright (c) 2021, PAL Robotics, S.L.
-All rights reserved.
-This work is licensed under the Creative Commons Attribution-NonCommercial-NoDerivs 3.0 Unported License.
-To view a copy of this license, visit http://creativecommons.org/licenses/by-nc-nd/3.0/ or send a letter to
-Creative Commons, 444 Castro Street, Suite 900, Mountain View, California, 94041, USA.
--->
+  Copyright (c) 2023 PAL Robotics S.L. All rights reserved.
+  Licensed under the Apache License, Version 2.0 (the "License");
+  you may not use this file except in compliance with the License.
+  You may obtain a copy of the License at
+      http://www.apache.org/licenses/LICENSE-2.0
+  Unless required by applicable law or agreed to in writing, software
+  distributed under the License is distributed on an "AS IS" BASIS,
+  WITHOUT WARRANTIES OR CONDITIONS OF ANY KIND, either express or implied.
+  See the License for the specific language governing permissions and
+  limitations under the License.
+ -->
 <robot xmlns:xacro="http://ros.org/wiki/xacro">
   <xacro:property name="PI" value="3.1415926535897931" />
-  <xacro:include filename="$(find omni_base_description)/urdf/wheels/wheel.transmission.xacro"/>
   <xacro:include filename="$(find omni_base_description)/urdf/wheels/wheel.gazebo.xacro"/>
   <!-- frontal_reflect: front: +1 and rear: -1 -->
@@ -83,7 +87,6 @@
       <axis xyz="0 0 1" />
       <limit effort="${torque}" velocity="${velocity / radius}"/>
+      <dynamics damping="1.0" friction="2.0"/>
     </joint>
-    <!-- Transmission -->
-    <xacro:wheel_transmission side="${side}"/>
     <!-- Gazebo extensions -->
     <xacro:wheel_gazebo side="${side}"/>

Commit message: ROS 2 omni base robot

File: omni_base_description/gazebo/gazebo.urdf.xacro (robot description, xacro)
@@ -31,13 +31,12 @@
       </xacro:unless>
     </plugin>
-    <!--@TODO: Migrate to humble, available in foxy-->
-    <!--<plugin filename="libgazebo_ros_force_based_move.so" name="gazebo_force_based_move" >
-      <commandTopic>mobile_base_controller/cmd_vel</commandTopic>
+    <plugin filename="libgazebo_ros_force_based_move.so" name="gazebo_force_based_move" >
+      <commandTopic>mobile_base_controller/cmd_vel_unstamped</commandTopic>
       <odometryTopic>mobile_base_controller/odom</odometryTopic>
       <odometryFrame>odom</odometryFrame>
       <odometryRate>50.0</odometryRate>
       <robotBaseFrame>base_footprint</robotBaseFrame>
-      <publishOdometryTf>true</publishOdometryTf>
-    </plugin>-->
+      <publishOdometryTf>false</publishOdometryTf>
+    </plugin>
   </gazebo>
   <gazebo reference="base_imu_link">

File: omni_base_description/robots/omni_base.urdf.xacro (robot description, xacro)
@@ -14,6 +14,6 @@
 <robot  xmlns:xacro="http://ros.org/wiki/xacro" name="omni_base" >
   <xacro:arg name="use_sim" default="true"/>
-  <xacro:arg name="front_laser_model" default="sick-571"/> <!-- false, hokuyo, sick-551, sick-561, sick-571-->
-  <xacro:arg name="rear_laser_model" default="sick-571"/> <!-- false, hokuyo, sick-551, sick-561, sick-571-->
+  <xacro:arg name="front_laser_model" default="sick-561"/> <!-- false, hokuyo, sick-551, sick-561, sick-571-->
+  <xacro:arg name="rear_laser_model" default="sick-561"/> <!-- false, hokuyo, sick-551, sick-561, sick-571-->
   <xacro:arg name="multiple" default="false"/>
   <xacro:arg name="namespace" default=""/>

File: omni_base_description/urdf/base/base_sensors.urdf.xacro (robot description, xacro)
@@ -9,8 +9,5 @@
 <robot xmlns:xacro="http://ros.org/wiki/xacro">
   <xacro:include filename="$(find omni_base_description)/urdf/base/base.urdf.xacro"/>
-  <xacro:include filename="$(find pmb2_description)/urdf/sensors/hokuyo_urg_04lx_ug01_laser.urdf.xacro"/>
-  <xacro:include filename="$(find pmb2_description)/urdf/sensors/sick_tim551_laser.urdf.xacro"/>
-  <xacro:include filename="$(find pmb2_description)/urdf/sensors/sick_tim561_laser.urdf.xacro"/>
-  <xacro:include filename="$(find pmb2_description)/urdf/sensors/sick_tim571_laser.urdf.xacro"/>
+  <xacro:include filename="$(find omni_base_description)/urdf/sensors/sick_tim561_laser.urdf.xacro"/>
   <xacro:include filename="$(find omni_base_description)/urdf/deg_to_rad.xacro"/>
   <!-- Laser model can be: false, hokuyo, sick-551, sick-561, sick-571-->
@@ -43,5 +40,5 @@
   <!-- front_laser_model can be: false, hokuyo, sick-551, sick-561, sick-571-->
   <!-- rear_laser_model can be: false, hokuyo, sick-551, sick-561, sick-571-->
-  <xacro:macro name="base_sensors" params=" name front_laser_model:=sick-571 rear_laser_model:=sick-571 laser_height:=0.13244">
+  <xacro:macro name="base_sensors" params=" name front_laser_model:=sick-561 rear_laser_model:=sick-561 laser_height:=0.13244">
     <!-- Rear Laser Sensor -->
     <xacro:laser_sensor name="${name}_rear_laser" parent="${name}" model="${rear_laser_model}" ros_topic="scan_rear_raw">
