Commit message: remove unused base_laser_link

File: omni_base_description/urdf/base/base_sensors.urdf.xacro (robot description, xacro)
@@ -44,26 +44,13 @@
   <!-- rear_left_laser_model can be: false, hokuyo, sick-551, sick-561, sick-571-->
   <xacro:macro name="base_sensors" params=" name front_right_laser_model:=sick-571 rear_left_laser_model:=sick-571">
-    <!-- Base Laser Link -->
-    <joint name="${name}_laser_joint" type="fixed">
-        <parent link="${name}_link"/>
-        <child link="${name}_laser_link"/>
-        <origin xyz="0 0 0.15614" rpy="0 0 0" />
-    </joint>
-    <link name="${name}_laser_link">
-        <inertial>
-            <origin xyz="0 0 0" rpy="0 0 0"/>
-            <mass value="0.0001" />
-            <inertia ixx="0.0001"  ixy="0"  ixz="0" iyy="0.0001" iyz="0" izz="0.0001" />
-        </inertial>
-    </link>
-    <!-- Rear Laser Sensor -->
-    <xacro:laser_sensor name="${name}_rear_laser" parent="${name}" model="${rear_left_laser_model}" ros_topic="scan_rear_raw">
-      <origin xyz="-0.27512 0.18297 0.13244" rpy="${-180 * deg_to_rad} 0 ${135 * deg_to_rad}" />
-    </xacro:laser_sensor>
-    <!-- Front Laser Sensor -->
-    <xacro:laser_sensor name="${name}_front_laser" parent="${name}" model="${front_right_laser_model}" ros_topic="scan_rear_raw">
-    <origin xyz="0.27512 -0.18297 0.13244" rpy="${-180 * deg_to_rad} 0 ${-45 * deg_to_rad}" />
-    </xacro:laser_sensor>
-    <xacro:base name="${name}"/>
+  <!-- Rear Laser Sensor -->
+  <xacro:laser_sensor name="${name}_rear_laser" parent="${name}" model="${rear_left_laser_model}" ros_topic="scan_rear_raw">
+    <origin xyz="-0.27512 0.18297 0.13244" rpy="${-180 * deg_to_rad} 0 ${135 * deg_to_rad}" />
+  </xacro:laser_sensor>
+  <!-- Front Laser Sensor -->
+  <xacro:laser_sensor name="${name}_front_laser" parent="${name}" model="${front_right_laser_model}" ros_topic="scan_rear_raw">
+  <origin xyz="0.27512 -0.18297 0.13244" rpy="${-180 * deg_to_rad} 0 ${-45 * deg_to_rad}" />
+  </xacro:laser_sensor>
+  <xacro:base name="${name}"/>
   </xacro:macro>
 </robot>

Commit message: added the virtual base laser link

File: omni_base_description/urdf/base/base_sensors.urdf.xacro (robot description, xacro)
@@ -44,14 +44,27 @@
   <!-- front_laser_model can be: false, hokuyo, sick-551, sick-561, sick-571-->
   <!-- rear_laser_model can be: false, hokuyo, sick-551, sick-561, sick-571-->
-  <xacro:macro name="base_sensors" params=" name front_laser_model:=sick-571 rear_laser_model:=sick-571">
-  <!-- Rear Laser Sensor -->
-  <xacro:laser_sensor name="${name}_rear_laser" parent="${name}" model="${rear_laser_model}" ros_topic="scan_rear_raw">
-    <origin xyz="-0.27512 0.18297 0.13244" rpy="${-180 * deg_to_rad} 0 ${135 * deg_to_rad}" />
-  </xacro:laser_sensor>
-  <!-- Front Laser Sensor -->
-  <xacro:laser_sensor name="${name}_front_laser" parent="${name}" model="${front_laser_model}" ros_topic="scan_front_raw">
-  <origin xyz="0.27512 -0.18297 0.13244" rpy="${-180 * deg_to_rad} 0 ${-45 * deg_to_rad}" />
-  </xacro:laser_sensor>
-  <xacro:base name="${name}"/>
+  <xacro:macro name="base_sensors" params=" name front_laser_model:=sick-571 rear_laser_model:=sick-571 laser_height:=0.13244">
+    <!-- Rear Laser Sensor -->
+    <xacro:laser_sensor name="${name}_rear_laser" parent="${name}" model="${rear_laser_model}" ros_topic="scan_rear_raw">
+      <origin xyz="-0.27512 0.18297 ${laser_height}" rpy="${-180 * deg_to_rad} 0 ${135 * deg_to_rad}" />
+    </xacro:laser_sensor>
+    <!-- Front Laser Sensor -->
+    <xacro:laser_sensor name="${name}_front_laser" parent="${name}" model="${front_laser_model}" ros_topic="scan_front_raw">
+    <origin xyz="0.27512 -0.18297 ${laser_height}" rpy="${-180 * deg_to_rad} 0 ${-45 * deg_to_rad}" />
+    </xacro:laser_sensor>
+    <!-- Virtual Base Laser Link -->
+    <joint name="virtual_${name}_laser_joint" type="fixed">
+        <parent link="${name}_link"/>
+        <child link="virtual_${name}_laser_link"/>
+        <origin xyz="0 0 ${laser_height}" rpy="0 0 0" />
+    </joint>
+    <link name="virtual_${name}_laser_link">
+        <inertial>
+            <origin xyz="0 0 0" rpy="0 0 0"/>
+            <mass value="0.0001" />
+            <inertia ixx="0.0001"  ixy="0"  ixz="0" iyy="0.0001" iyz="0" izz="0.0001" />
+        </inertial>
+    </link>
+    <xacro:base name="${name}"/>
   </xacro:macro>
 </robot>

Commit message: fix the min and max angle of the lasers

File: omni_base_description/urdf/base/base_sensors.urdf.xacro (robot description, xacro)
@@ -16,5 +16,5 @@
   <!-- Laser model can be: false, hokuyo, sick-551, sick-561, sick-571-->
   <!-- Laser:  Theoretic FOV = 220 -->
-  <xacro:macro name="laser_sensor" params="name parent model ros_topic *origin update_rate:=10 min_angle:=${-110 * deg_to_rad} max_angle:=${110 * deg_to_rad}">
+  <xacro:macro name="laser_sensor" params="name parent model ros_topic *origin min_angle max_angle update_rate:=10">
     <xacro:if value="${model == 'sick-551'}">
       <!-- Rear Laser:  Theoretic FOV = 220 -->
@@ -46,9 +46,9 @@
   <xacro:macro name="base_sensors" params=" name front_laser_model:=sick-571 rear_laser_model:=sick-571 laser_height:=0.13244">
     <!-- Rear Laser Sensor -->
-    <xacro:laser_sensor name="${name}_rear_laser" parent="${name}" model="${rear_laser_model}" ros_topic="scan_rear_raw">
+    <xacro:laser_sensor name="${name}_rear_laser" parent="${name}" model="${rear_laser_model}" ros_topic="scan_rear_raw" min_angle="${-110 * deg_to_rad}" max_angle="${110 * deg_to_rad}">
       <origin xyz="-0.27512 0.18297 ${laser_height}" rpy="${-180 * deg_to_rad} 0 ${135 * deg_to_rad}" />
     </xacro:laser_sensor>
     <!-- Front Laser Sensor -->
-    <xacro:laser_sensor name="${name}_front_laser" parent="${name}" model="${front_laser_model}" ros_topic="scan_front_raw">
+    <xacro:laser_sensor name="${name}_front_laser" parent="${name}" model="${front_laser_model}" ros_topic="scan_front_raw" min_angle="${-110 * deg_to_rad}" max_angle="${110 * deg_to_rad}">
     <origin xyz="0.27512 -0.18297 ${laser_height}" rpy="${-180 * deg_to_rad} 0 ${-45 * deg_to_rad}" />
     </xacro:laser_sensor>

Commit message: fix laser fov for omni base

File: omni_base_description/urdf/base/base_sensors.urdf.xacro (robot description, xacro)
@@ -15,27 +15,26 @@
   <xacro:include filename="$(find omni_base_description)/urdf/deg_to_rad.xacro"/>
   <!-- Laser model can be: false, hokuyo, sick-551, sick-561, sick-571-->
-  <!-- Laser:  Theoretic FOV = 220 -->
-  <xacro:macro name="laser_sensor" params="name parent model ros_topic *origin min_angle max_angle update_rate:=10">
+  <xacro:macro name="laser_sensor" params="name parent model ros_topic *origin update_rate:=10">
     <xacro:if value="${model == 'sick-551'}">
-      <!-- Rear Laser:  Theoretic FOV = 220 -->
-      <xacro:sick_tim551_laser name="${name}" parent="${parent}" ros_topic="${ros_topic}" update_rate="${update_rate}" min_angle="${min_angle}" max_angle="${max_angle}" >
+      <!-- Rear Laser:  Theoretic FOV = 270 -->
+      <xacro:sick_tim551_laser name="${name}" parent="${parent}" ros_topic="${ros_topic}" update_rate="${update_rate}" min_angle="${-135 * deg_to_rad}" max_angle="${135 * deg_to_rad}" >
         <xacro:insert_block name="origin" />
       </xacro:sick_tim551_laser>
     </xacro:if>
     <xacro:if value="${model == 'sick-561'}">
-      <!-- Rear Laser:  Theoretic FOV = 220 -->
-      <xacro:sick_tim561_laser name="${name}" parent="${parent}" ros_topic="${ros_topic}" update_rate="${update_rate}" min_angle="${min_angle}" max_angle="${max_angle}" >
+      <!-- Rear Laser:  Theoretic FOV = 270 -->
+      <xacro:sick_tim561_laser name="${name}" parent="${parent}" ros_topic="${ros_topic}" update_rate="${update_rate}" min_angle="${-135 * deg_to_rad}" max_angle="${135 * deg_to_rad}" >
         <xacro:insert_block name="origin" />
       </xacro:sick_tim561_laser>
     </xacro:if>
     <xacro:if value="${model == 'sick-571'}">
-      <!-- Rear Laser:  Theoretic FOV = 220 -->
-      <xacro:sick_tim571_laser name="${name}" parent="${parent}" ros_topic="${ros_topic}" update_rate="${update_rate}" min_angle="${min_angle}" max_angle="${max_angle}" >
+      <!-- Rear Laser:  Theoretic FOV = 270 -->
+      <xacro:sick_tim571_laser name="${name}" parent="${parent}" ros_topic="${ros_topic}" update_rate="${update_rate}" min_angle="${-135 * deg_to_rad}" max_angle="${135 * deg_to_rad}" >
         <xacro:insert_block name="origin" />
       </xacro:sick_tim571_laser>
     </xacro:if>
     <xacro:if value="${model == 'hokuyo'}">
-      <!-- Rear Laser:  Theoretic FOV = 220 -->
-      <xacro:hokuyo_urg_04lx_ug01_laser name="${name}" parent="${parent}" ros_topic="${ros_topic}" update_rate="${update_rate}" min_angle="${min_angle}" max_angle="${max_angle}" >
+      <!-- Rear Laser:  Theoretic FOV = 240 -->
+      <xacro:hokuyo_urg_04lx_ug01_laser name="${name}" parent="${parent}" ros_topic="${ros_topic}" update_rate="${update_rate}" min_angle="${-120 * deg_to_rad}" max_angle="${120 * deg_to_rad}" >
         <xacro:insert_block name="origin" />
       </xacro:hokuyo_urg_04lx_ug01_laser>
@@ -46,10 +45,10 @@
   <xacro:macro name="base_sensors" params=" name front_laser_model:=sick-571 rear_laser_model:=sick-571 laser_height:=0.13244">
     <!-- Rear Laser Sensor -->
-    <xacro:laser_sensor name="${name}_rear_laser" parent="${name}" model="${rear_laser_model}" ros_topic="scan_rear_raw" min_angle="${-110 * deg_to_rad}" max_angle="${110 * deg_to_rad}">
+    <xacro:laser_sensor name="${name}_rear_laser" parent="${name}" model="${rear_laser_model}" ros_topic="scan_rear_raw">
       <origin xyz="-0.27512 0.18297 ${laser_height}" rpy="${-180 * deg_to_rad} 0 ${135 * deg_to_rad}" />
     </xacro:laser_sensor>
     <!-- Front Laser Sensor -->
-    <xacro:laser_sensor name="${name}_front_laser" parent="${name}" model="${front_laser_model}" ros_topic="scan_front_raw" min_angle="${-110 * deg_to_rad}" max_angle="${110 * deg_to_rad}">
-    <origin xyz="0.27512 -0.18297 ${laser_height}" rpy="${-180 * deg_to_rad} 0 ${-45 * deg_to_rad}" />
+    <xacro:laser_sensor name="${name}_front_laser" parent="${name}" model="${front_laser_model}" ros_topic="scan_front_raw">
+      <origin xyz="0.27512 -0.18297 ${laser_height}" rpy="${-180 * deg_to_rad} 0 ${-45 * deg_to_rad}" />
     </xacro:laser_sensor>
     <!-- Virtual Base Laser Link -->

Commit message: Change path related to restructure path for pal_urdf_utils

File: omni_base_description/urdf/base/base_sensors.urdf.xacro (robot description, xacro)
@@ -15,9 +15,9 @@
   <!-- INCLUDES -->
   <xacro:include filename="$(find omni_base_description)/urdf/base/base.urdf.xacro"/>
-  <xacro:include filename="$(find pal_urdf_utils)/urdf/sensors/imu.urdf.xacro"/>
-  <xacro:include filename="$(find pal_urdf_utils)/urdf/sensors/hokuyo_urg_04lx_ug01_laser.urdf.xacro"/>
-  <xacro:include filename="$(find pal_urdf_utils)/urdf/sensors/bases/sick_tim551_laser.urdf.xacro"/>
-  <xacro:include filename="$(find pal_urdf_utils)/urdf/sensors/bases/sick_tim561_laser.urdf.xacro"/>
-  <xacro:include filename="$(find pal_urdf_utils)/urdf/sensors/bases/sick_tim571_laser.urdf.xacro"/>
+  <xacro:include filename="$(find pal_urdf_utils)/urdf/interaction_sensors/imu.urdf.xacro"/>
+  <xacro:include filename="$(find pal_urdf_utils)/urdf/laser/hokuyo_urg_04lx_ug01_laser.urdf.xacro"/>
+  <xacro:include filename="$(find pal_urdf_utils)/urdf/laser/sick_tim551_laser.urdf.xacro"/>
+  <xacro:include filename="$(find pal_urdf_utils)/urdf/laser/sick_tim561_laser.urdf.xacro"/>
+  <xacro:include filename="$(find pal_urdf_utils)/urdf/laser/sick_tim571_laser.urdf.xacro"/>
   <!-- LASER MACRO DEFINITION -->
   <xacro:macro name="laser_sensor" params="name parent model ros_topic *origin update_rate:=10">

File: omni_base_description/urdf/cameras_add_on/cameras.urdf.xacro (robot description, xacro)
@@ -26,7 +26,12 @@
   <xacro:property name="roof_rgbd_y" value="0.0"/>
   <xacro:property name="roof_rgbd_Y" value="0.0"/>
-  <!-- base/roof RGBD calibratable characteristics -->
-  <!-- spec = rgbd_z, rgbd_R and rgbd_P -->
-  <xacro:include filename="${calibration_path}/urdf/cameras_add_on/base_omni_base_calib.urdf.xacro"/>
+  <!-- RGBD base -->
+  <xacro:property name="base_rgbd_z" value="0.551436"/>
+  <xacro:property name="base_rgbd_R" value="0.0"/>
+  <xacro:property name="base_rgbd_P" value="55.0"/>
+  <!-- RGBD roof -->
+  <xacro:property name="roof_rgbd_z" value="0.483197"/>
+  <xacro:property name="roof_rgbd_R" value="0.0"/>
+  <xacro:property name="roof_rgbd_P" value="12.0"/>
   <xacro:include filename="$(find pal_urdf_utils)/urdf/deg_to_rad.urdf.xacro" />
   <xacro:if value="${camera_model == 'realsense-d435'}">
