Commit message: Changed laser scan topic for the simulation navigation

File: omni_base_description/urdf/base/base.urdf.xacro (robot description, xacro)
@@ -27,5 +27,5 @@
           iyy="0.462761159488672" iyz="0.00110342934873762" izz="0.454645990122976" />
       </inertial>
-      <visual>
+      <!-- <visual>
         <origin xyz="0 0 0" rpy="0 0 0" />
         <geometry>
@@ -41,5 +41,5 @@
           <mesh filename="package://omni_base_description/meshes/base/base_link.dae" />
         </geometry>
-      </collision>
+      </collision> -->
     </link>
     <link name="${name}_footprint"/>

File: omni_base_description/urdf/base/base_sensors.urdf.xacro (robot description, xacro)
@@ -26,8 +26,8 @@
     </link>
     <!-- Rear Laser:  Theoretic FOV = 220 -->
-    <xacro:sick_tim561_laser name="${name}_rear_laser" parent="${name}" ros_topic="scan_rear" update_rate="10" min_angle="${-120 * deg_to_rad}" max_angle="${120 * deg_to_rad}"  >
+    <xacro:sick_tim561_laser name="${name}_rear_laser" parent="${name}" ros_topic="scan_rear_raw" update_rate="10" min_angle="${-120 * deg_to_rad}" max_angle="${120 * deg_to_rad}"  >
       <origin xyz="-0.277 0 0.15614" rpy="0 0 ${180 * deg_to_rad}" />
     </xacro:sick_tim561_laser>
-    <xacro:sick_tim561_laser name="${name}_front_laser" parent="${name}" ros_topic="scan_front" update_rate="10" min_angle="${-120 * deg_to_rad}" max_angle="${120 * deg_to_rad}" >
+    <xacro:sick_tim561_laser name="${name}_front_laser" parent="${name}" ros_topic="scan_front_raw" update_rate="10" min_angle="${-120 * deg_to_rad}" max_angle="${120 * deg_to_rad}" >
       <origin xyz="0.277 0 0.15614" rpy="0 0 0" />
     </xacro:sick_tim561_laser>

Commit message: update the base_link mesh and the link information

File: omni_base_description/urdf/base/base.urdf.xacro (robot description, xacro)
@@ -22,10 +22,10 @@
     <link name="${name}_link">
       <inertial>
-        <origin xyz="-0.00714862613301571 -0.00611949538965259 0.17932103073575" rpy="0 0 0" />
-        <mass value="40.5916085964121" />
-        <inertia ixx="0.347483846337784" ixy="0.00017011926290181" ixz="-0.00450619609287122"
-          iyy="0.462761159488672" iyz="0.00110342934873762" izz="0.454645990122976" />
+        <origin xyz="0.0026742 0.00027459 0.086363" rpy="0 0 0" />
+        <mass value="34.047" />
+        <inertia ixx="0.22777" ixy="0.00035979" ixz="0.00015269"
+          iyy="0.29991" iyz="1.7872E-05" izz="0.46036" />
       </inertial>
-      <!-- <visual>
+      <visual>
         <origin xyz="0 0 0" rpy="0 0 0" />
         <geometry>
@@ -33,5 +33,5 @@
         </geometry>
         <material name="">
-          <color rgba="0.250980392156863 0.250980392156863 0.250980392156863 1" />
+          <color rgba="0.75294 0.75294 0.75294 1" />
         </material>
       </visual>
@@ -41,5 +41,5 @@
           <mesh filename="package://omni_base_description/meshes/base/base_link.dae" />
         </geometry>
-      </collision> -->
+      </collision>
     </link>
     <link name="${name}_footprint"/>
@@ -49,5 +49,5 @@
       <parent link="${name}_footprint"/>
     </joint>
-  <!-- gazebo parameters are given here for base_link thru base_footprint -->
+  <!-- gazebo parameters are given here for base_link through base_footprint -->
     <gazebo reference="${name}_footprint">
       <kp>100000000.0</kp>
@@ -62,5 +62,5 @@
     <!-- IMU -->
     <xacro:imu_sensor name="${name}_imu" parent="${name}_link" update_rate="100.0">
-      <origin xyz="-0.229392176792506 0 0.0788684081014052" rpy="${-70 * deg_to_rad} 0 ${90 * deg_to_rad}"/>
+      <origin xyz="-0.287 0 0.092163" rpy="0 0 ${90.0 * deg_to_rad}" />
     </xacro:imu_sensor>
     <xacro:wheel side="front_right" reflect=" 1.0" radius="${wheel_radius}" width="${wheel_width}" torque="${wheel_torque}" velocity="${wheel_velocity}" pair_separation="${wheel_pair_separation}"  separation="${wheel_separation}" parent="${name}"/>

Commit message: update the wheel separation, radius and width parameters

File: omni_base_description/urdf/base/base.urdf.xacro (robot description, xacro)
@@ -12,8 +12,8 @@
   <xacro:include filename="$(find pmb2_description)/urdf/sensors/imu.urdf.xacro"/>
   <!-- Wheel characteristics -->
-  <xacro:property name="wheel_radius"     value="0.1016"/>
-  <xacro:property name="wheel_width"      value="0.078"/>
-  <xacro:property name="wheel_separation" value="0.526"/>
-  <xacro:property name="wheel_pair_separation" value="0.410"/>
+  <xacro:property name="wheel_radius"     value="0.0762"/>
+  <xacro:property name="wheel_width"      value="0.050"/>
+  <xacro:property name="wheel_separation" value="0.44715"/>
+  <xacro:property name="wheel_pair_separation" value="0.488"/>
   <xacro:property name="wheel_torque"     value="6.0"/>
   <xacro:property name="wheel_velocity"   value="1.0"/>

Commit message: added antenna's links and meshes

File: omni_base_description/urdf/base/base.urdf.xacro (robot description, xacro)
@@ -10,4 +10,5 @@
   <xacro:include filename="$(find omni_base_description)/urdf/deg_to_rad.xacro"/>
   <xacro:include filename="$(find omni_base_description)/urdf/wheels/wheel.urdf.xacro"/>
+  <xacro:include filename="$(find omni_base_description)/urdf/base/antenna.urdf.xacro"/>
   <xacro:include filename="$(find pmb2_description)/urdf/sensors/imu.urdf.xacro"/>
   <!-- Wheel characteristics -->
@@ -64,4 +65,11 @@
       <origin xyz="-0.287 0 0.092163" rpy="0 0 ${90.0 * deg_to_rad}" />
     </xacro:imu_sensor>
+    <!-- Antennas -->
+    <xacro:antenna name="base_antena_right" parent="base_link" reflect="1">
+      <origin xyz="-0.2015 -0.13 0.2165" rpy="0 0 0" />
+    </xacro:antenna>
+    <xacro:antenna name="base_antena_left" parent="base_link" reflect="-1">
+      <origin xyz="-0.2015 0.13 0.2165" rpy="0 0 0" />
+    </xacro:antenna>
     <xacro:wheel side="front_right" reflect=" 1.0" radius="${wheel_radius}" width="${wheel_width}" torque="${wheel_torque}" velocity="${wheel_velocity}" pair_separation="${wheel_pair_separation}"  separation="${wheel_separation}" parent="${name}"/>
     <xacro:wheel side="front_left"  reflect="-1.0" radius="${wheel_radius}" width="${wheel_width}" torque="${wheel_torque}" velocity="${wheel_velocity}" pair_separation="${wheel_pair_separation}"  separation="${wheel_separation}" parent="${name}"/>

Commit message: added base docking link frame

File: omni_base_description/urdf/base/base.urdf.xacro (robot description, xacro)
@@ -65,4 +65,34 @@
       <origin xyz="-0.287 0 0.092163" rpy="0 0 ${90.0 * deg_to_rad}" />
     </xacro:imu_sensor>
+    <!-- Docking link -->
+    <link name="${name}_dock_link">
+      <inertial>
+        <origin xyz="-0.0037082 1.5226E-18 -4.1633E-17" rpy="0 0 0" />
+        <mass value="0.032242" />
+        <inertia ixx="2.1302E-05" ixy="-1.0461E-21" ixz="6.6555E-22"
+          iyy="1.2058E-05" iyz="-1.9453E-21" izz="1.0058E-05" />
+      </inertial>
+      <visual>
+        <origin xyz="0 0 0" rpy="0 0 0" />
+        <geometry>
+          <mesh filename="package://omni_base_description/meshes/base/base_dock_link.stl" />
+        </geometry>
+        <material name="">
+          <color rgba="0.25098 0.25098 0.25098 1" />
+        </material>
+      </visual>
+      <collision>
+        <origin xyz="0 0 0" rpy="0 0 0" />
+        <geometry>
+          <mesh filename="package://omni_base_description/meshes/base/base_dock_link.stl" />
+        </geometry>
+      </collision>
+    </link>
+    <joint name="${name}_dock" type="fixed">
+      <origin xyz="0.3535 0 0.0596" rpy="0 0 0" />
+      <parent link="${name}_link" />
+      <child link="${name}_dock_link" />
+      <axis xyz="0 0 0" />
+    </joint>
     <!-- Antennas -->
     <xacro:antenna name="base_antena_right" parent="base_link" reflect="1">

Commit message: update the new wheel macro in the main URDF

File: omni_base_description/urdf/base/base.urdf.xacro (robot description, xacro)
@@ -19,4 +19,5 @@
   <xacro:property name="wheel_torque"     value="6.0"/>
   <xacro:property name="wheel_velocity"   value="1.0"/>
+  <xacro:property name="suspension_sagital_separation" value="0.345"/>
   <xacro:macro name="base" params="name">
     <!-- Base footprint -->
@@ -102,8 +103,8 @@
       <origin xyz="-0.2015 0.13 0.2165" rpy="0 0 0" />
     </xacro:antenna>
-    <xacro:wheel side="front_right" reflect=" 1.0" radius="${wheel_radius}" width="${wheel_width}" torque="${wheel_torque}" velocity="${wheel_velocity}" pair_separation="${wheel_pair_separation}"  separation="${wheel_separation}" parent="${name}"/>
-    <xacro:wheel side="front_left"  reflect="-1.0" radius="${wheel_radius}" width="${wheel_width}" torque="${wheel_torque}" velocity="${wheel_velocity}" pair_separation="${wheel_pair_separation}"  separation="${wheel_separation}" parent="${name}"/>
-    <xacro:wheel side="back_right"  reflect=" 1.0" radius="${wheel_radius}" width="${wheel_width}" torque="${wheel_torque}" velocity="${wheel_velocity}" pair_separation="${-wheel_pair_separation}" separation="${wheel_separation}" parent="${name}"/>
-    <xacro:wheel side="back_left"   reflect="-1.0" radius="${wheel_radius}" width="${wheel_width}" torque="${wheel_torque}" velocity="${wheel_velocity}" pair_separation="${-wheel_pair_separation}" separation="${wheel_separation}" parent="${name}"/>
+    <xacro:wheel side="front_right" sagital_reflect="1.0" frontal_reflect="1.0" radius="${wheel_radius}" width="${wheel_width}" torque="${wheel_torque}" velocity="${wheel_velocity}" frontal_separation="${wheel_pair_separation}"  sagital_separation="${suspension_sagital_separation}" parent="${name}_link"/>
+    <xacro:wheel side="front_left"  sagital_reflect="-1.0" frontal_reflect="1.0" radius="${wheel_radius}" width="${wheel_width}" torque="${wheel_torque}" velocity="${wheel_velocity}" frontal_separation="${wheel_pair_separation}"  sagital_separation="${suspension_sagital_separation}" parent="${name}_link"/>
+    <xacro:wheel side="rear_right"  sagital_reflect="1.0" frontal_reflect="-1.0" radius="${wheel_radius}" width="${wheel_width}" torque="${wheel_torque}" velocity="${wheel_velocity}" frontal_separation="${wheel_pair_separation}" sagital_separation="${suspension_sagital_separation}" parent="${name}_link"/>
+    <xacro:wheel side="rear_left"   sagital_reflect="-1.0" frontal_reflect="-1.0" radius="${wheel_radius}" width="${wheel_width}" torque="${wheel_torque}" velocity="${wheel_velocity}" frontal_separation="${wheel_pair_separation}" sagital_separation="${suspension_sagital_separation}" parent="${name}_link"/>
   </xacro:macro>
 </robot>

Commit message: Update the collision model of the base_link

File: omni_base_description/urdf/base/base.urdf.xacro (robot description, xacro)
@@ -39,7 +39,7 @@
       </visual>
       <collision>
-        <origin xyz="0 0 0" rpy="0 0 0" />
+        <origin xyz="0 0 0.0925" rpy="0 0 0" />
         <geometry>
-          <mesh filename="package://omni_base_description/meshes/base/base_link.dae" />
+          <box size="0.75 0.5 0.275"/>
         </geometry>
       </collision>

Commit message: Split the collision into 2 boxes for the sake of laser

File: omni_base_description/urdf/base/base.urdf.xacro (robot description, xacro)
@@ -39,7 +39,13 @@
       </visual>
       <collision>
-        <origin xyz="0 0 0.0925" rpy="0 0 0" />
+        <origin xyz="0 0 0.185" rpy="0 0 0" />
         <geometry>
-          <box size="0.75 0.5 0.275"/>
+          <box size="0.72 0.5 0.08"/>
+        </geometry>
+      </collision>
+      <collision>
+        <origin xyz="0 0 0.04" rpy="0 0 0" />
+        <geometry>
+          <box size="0.72 0.5 0.17"/>
         </geometry>
       </collision>

Commit message: Using the full mesh instead of the two boxes

File: omni_base_description/urdf/base/base.urdf.xacro (robot description, xacro)
@@ -39,13 +39,7 @@
       </visual>
       <collision>
-        <origin xyz="0 0 0.185" rpy="0 0 0" />
+        <origin xyz="0 0 0" rpy="0 0 0" />
         <geometry>
-          <box size="0.72 0.5 0.08"/>
-        </geometry>
-      </collision>
-      <collision>
-        <origin xyz="0 0 0.04" rpy="0 0 0" />
-        <geometry>
-          <box size="0.72 0.5 0.17"/>
+          <mesh filename="package://omni_base_description/meshes/base/base_link.stl" />
         </geometry>
       </collision>

Commit message: Fix collision boxes for the base

File: omni_base_description/urdf/base/base.urdf.xacro (robot description, xacro)
@@ -39,7 +39,19 @@
       </visual>
       <collision>
-        <origin xyz="0 0 0" rpy="0 0 0" />
+        <origin xyz="0 0 0.18925" rpy="0 0 0" />
         <geometry>
-          <mesh filename="package://omni_base_description/meshes/base/base_link.stl" />
+          <box size="0.717 0.497 0.0845"/>
+        </geometry>
+      </collision>
+      <collision>
+        <origin xyz="0 0 0.132" rpy="0 0 0" />
+        <geometry>
+          <box size="0.58 0.39 0.03"/>
+        </geometry>
+      </collision>
+      <collision>
+        <origin xyz="0 0 0.04" rpy="0 0 0" />
+        <geometry>
+          <box size="0.715 0.48 0.154"/>
         </geometry>
       </collision>

Commit message: Update box dimensions

File: omni_base_description/urdf/base/base.urdf.xacro (robot description, xacro)
@@ -51,7 +51,7 @@
       </collision>
       <collision>
-        <origin xyz="0 0 0.04" rpy="0 0 0" />
+        <origin xyz="0 0 0.0335" rpy="0 0 0" />
         <geometry>
-          <box size="0.715 0.48 0.154"/>
+          <box size="0.705 0.48 0.167"/>
         </geometry>
       </collision>

Commit message: Increase Wheel max velocity

File: omni_base_description/urdf/base/base.urdf.xacro (robot description, xacro)
@@ -20,5 +20,6 @@
   <xacro:property name="wheel_pair_separation" value="0.488"/>
   <xacro:property name="wheel_torque"     value="6.0"/>
-  <xacro:property name="wheel_velocity"   value="1.0"/>
+  <!-- To Do: Compute real wheel max velocity -->
+  <xacro:property name="wheel_velocity"   value="10.0"/>
   <xacro:property name="suspension_sagital_separation" value="0.345"/>
   <!-- INCLUDES -->

File: omni_base_description/urdf/wheels/wheel.ros2_control.xacro (robot description, xacro)
@@ -17,6 +17,7 @@
     <joint name="wheel_${side}_joint">
       <command_interface name="velocity">
-        <param name="min">-1</param>
-        <param name="max">1</param>
+        <!-- To Do: Compute real wheel max velocity -->
+        <param name="min">-10</param>
+        <param name="max">10</param>
       </command_interface>
       <state_interface name="position" />

Commit message: increase max an min vel

File: omni_base_description/urdf/base/base.urdf.xacro (robot description, xacro)
@@ -21,5 +21,5 @@
   <xacro:property name="wheel_torque"     value="6.0"/>
   <!-- TODO Compute real wheel max velocity -->
-  <xacro:property name="wheel_velocity"   value="10.0"/>
+  <xacro:property name="wheel_velocity"   value="100.0"/>
   <xacro:property name="suspension_sagital_separation" value="0.345"/>
   <!-- INCLUDES -->

File: omni_base_description/urdf/wheels/wheel.ros2_control.xacro (robot description, xacro)
@@ -18,6 +18,6 @@
     <joint name="wheel_${side}_joint">
       <command_interface name="velocity">
-        <param name="min">-10</param>
-        <param name="max">10</param>
+        <param name="min">-100</param>
+        <param name="max">100</param>
       </command_interface>
       <state_interface name="position" />
