Commit message: added mesh and position of camera on top

File: omni_base_description/urdf/cameras_add_on/camera_on_top.urdf.xacro (robot description, xacro)
@@ -17,6 +17,6 @@
     <link name="${name}_link">
       <inertial>
-        <origin xyz="-0.00001132 0.04392363 0.06783541" rpy="0.0 0.0 0.0"/>
-        <mass value="3.057"/>
+        <origin xyz="0 0 0" rpy="0 0 0"/>
+        <mass value="0.1"/>
         <inertia ixx="0.08241443" ixy="-0.00000558" ixz="-0.00001319"
           iyy="0.05540468" iyz="0.01732357"
@@ -24,5 +24,5 @@
         </inertial>
         <visual>
-          <origin xyz="0 0 -0.04" rpy="1.57 0 1.57"/>
+          <origin xyz="0 0 0" rpy="0 0 0"/>
           <geometry>
             <mesh filename="package://omni_base_description/meshes/cameras_add_on/camera_on_top.stl" scale="1 1 1"/>
@@ -31,5 +31,5 @@
         </visual>
         <collision>
-          <origin xyz="0 0 -0.04" rpy="1.57 0 1.57"/>
+          <origin xyz="0 0 0" rpy="0 0 0"/>
           <geometry>
             <mesh filename="package://omni_base_description/meshes/cameras_add_on/camera_on_top.stl" scale="1 1 1"/>

File: omni_base_description/urdf/sensors/camera_on_top.urdf.xacro (robot description, xacro)
@@ -13,25 +13,13 @@
 -->
 <robot xmlns:xacro="http://ros.org/wiki/xacro">
-  <!-- PROPERTIES -->
   <!-- Execution env config -->
-  <xacro:property name="default_calibration_path" value="$(find omni_base_description)"/>
-  <xacro:property name="calibration_path" value="$(optenv omni_base_description_calibration_path ${default_calibration_path})"/>
   <xacro:property name="use_sim_time" value="$(arg use_sim_time)" />
-  <!-- base RGBD characteristics -->
-  <xacro:property name="base_rgbd_x" value="0.327327"/>
-  <xacro:property name="base_rgbd_y" value="0.0"/>
-  <xacro:property name="base_rgbd_Y" value="0.0"/>
-  <!-- roof RGBD characteristics -->
-  <xacro:property name="roof_rgbd_x" value="0.297329"/>
-  <xacro:property name="roof_rgbd_y" value="0.0"/>
-  <xacro:property name="roof_rgbd_Y" value="0.0"/>
-  <!-- base/roof RGBD calibratable characteristics -->
-  <!-- spec = rgbd_z, rgbd_R and rgbd_P -->
-  <xacro:include filename="${calibration_path}/urdf/cameras_add_on/base_omni_base_calib.urdf.xacro"/>
+  <!--RGBD characteristics -->
+  <xacro:property name="rgbd_x" value="0.28595"/>
+  <xacro:property name="rgbd_y" value="0.0"/>
+  <xacro:property name="rgbd_z" value="0.28125"/>
   <xacro:include filename="$(find pal_urdf_utils)/urdf/deg_to_rad.urdf.xacro" />
   <xacro:if value="${camera_model == 'realsense-d435'}">
-    <!-- INCLUDES -->
     <xacro:include filename="$(find realsense2_description)/urdf/_d435.urdf.xacro" />
-    <!-- RGBD base -->
     <xacro:sensor_d435
       name="rgbd_camera"
@@ -40,15 +28,12 @@
       use_nominal_extrinsics="${use_sim_time}">
       <origin
-          xyz="${base_rgbd_x}
-              ${base_rgbd_y}
-              ${base_rgbd_z}"
-          rpy="${base_rgbd_R * deg_to_rad}
-              ${base_rgbd_P * deg_to_rad}
-              ${base_rgbd_Y * deg_to_rad}"/>
+          xyz="${rgbd_x}
+              ${rgbd_y}
+              ${rgbd_z}"
+          rpy="0.0 0.0 0.0"/>
     </xacro:sensor_d435>
+  </xacro:if>
   <xacro:if value="${camera_model == 'realsense-d435i'}">
-    <!-- INCLUDES -->
     <xacro:include filename="$(find realsense2_description)/urdf/_d435i.urdf.xacro" />
-    <!-- RGBD base -->
     <xacro:sensor_d435i
       name="rgbd_camera"
@@ -57,10 +42,9 @@
       use_nominal_extrinsics="${use_sim_time}">
       <origin
-          xyz="${base_rgbd_x}
-              ${base_rgbd_y}
-              ${base_rgbd_z}"
-          rpy="${base_rgbd_R * deg_to_rad}
-              ${base_rgbd_P * deg_to_rad}
-              ${base_rgbd_Y * deg_to_rad}"/>
+          xyz="${rgbd_x}
+              ${rgbd_y}
+              ${rgbd_z}"
+          rpy="0.0 0.0 0.0"/>
     </xacro:sensor_d435i>
+  </xacro:if>
 </robot>
