Commit message: update inertia

File: omni_base_description/urdf/cameras_add_on/camera_horizon_add_on.urdf.xacro (robot description, xacro)
@@ -24,7 +24,7 @@
         <origin xyz="0 0 0" rpy="0 0 0"/>
         <mass value="0.1"/>
-        <inertia ixx="0.08241443" ixy="-0.00000558" ixz="-0.00001319"
-          iyy="0.05540468" iyz="0.01732357"
-          izz="0.07634613"/>
+        <inertia ixx="0.00009667" ixy="0.0" ixz="0.0"
+          iyy="0.0" iyz="0.0"
+          izz="0.00027083"/>
         </inertial>
         <visual>
