Commit message: add gazebo versioning parameters

File: omni_base_description/ros2_control/ros2_control.urdf.xacro (robot description, xacro)
@@ -20,14 +20,25 @@
     <xacro:if value="${use_sim_time}">
       <gazebo>
-        <plugin filename="libgazebo_ros2_control.so" name="gazebo_ros2_control">
-          <ros>
-            <namespace>${namespace}</namespace>
-            <remapping>/tf:=tf</remapping>
-            <remapping>/tf_static:=tf_static</remapping>
-          </ros>
-          <parameters>$(find omni_base_description)/ros2_control/gazebo_controller_manager_cfg.yaml</parameters>
-          <!-- <robot_sim_type>gazebo_ros2_control/GazeboSystem</robot_sim_type>
-          <control_period>0.001</control_period> -->
-        </plugin>
+        <xacro:if value="${gazebo_version == 'classic'}">
+          <plugin filename="libgazebo_ros2_control.so" name="gazebo_ros2_control">
+            <ros>
+              <namespace>${namespace}</namespace>
+              <remapping>/tf:=tf</remapping>
+              <remapping>/tf_static:=tf_static</remapping>
+            </ros>
+            <parameters>$(find stockbot_description)/ros2_control/gazebo_controller_manager_cfg.yaml</parameters>
+          </plugin>
+        </xacro:if>
+        <xacro:if value="${gazebo_version == 'gazebo'}">
+          <plugin filename="gz_ros2_control-system" name="gz_ros2_control::GazeboSimROS2ControlPlugin">
+            <parameters>$(find omni_base_description)/ros2_control/gazebo_controller_manager_cfg.yaml</parameters>
+            <robot_param>robot_description</robot_param>
+            <robot_param_node>robot_state_publisher</robot_param_node>
+            <ros>
+              <remapping>/mecanum_drive_controller/reference:=/cmd_vel</remapping>
+              <remapping>/mecanum_drive_controller/odom:=/odom</remapping>
+            </ros>
+          </plugin>
+        </xacro:if>
       </gazebo>
     </xacro:if>
@@ -38,5 +49,10 @@
         <!-- HW interface; gazebo-->
         <hardware>
-          <plugin>gazebo_ros2_control/GazeboSystem</plugin>
+          <xacro:if value="${gazebo_version == 'classic'}">
+            <plugin>gazebo_ros2_control/GazeboSystem</plugin>
+          </xacro:if>
+          <xacro:if value="${gazebo_version == 'gazebo'}">
+            <plugin>gz_ros2_control/GazeboSimSystem</plugin>
+          </xacro:if>
         </hardware>
       </xacro:if>
@@ -44,5 +60,10 @@
         <!-- HW interface; robot control-->
         <hardware>
-          <plugin>robot_control/RobotControl</plugin>
+          <xacro:if value="${gazebo_version == 'classic'}">
+            <plugin>gazebo_ros2_control/GazeboSystem</plugin>
+          </xacro:if>
+          <xacro:if value="${gazebo_version == 'gazebo'}">
+            <plugin>gz_ros2_control/GazeboSimSystem</plugin>
+          </xacro:if>
         </hardware>
       </xacro:unless>

File: omni_base_description/urdf/base/base.gazebo.xacro (robot description, xacro)
@@ -31,4 +31,5 @@
     </gazebo>
     <!-- Odometry plugin for ground truth -->
+  <xacro:if value="${gazebo_version == 'classic'}">
     <gazebo>
       <plugin name="gazebo_ros_planar_move" filename="libgazebo_ros_planar_move.so">
@@ -54,4 +55,5 @@
       </plugin>
     </gazebo>
+  </xacro:if>
   </xacro:macro>
 </robot>

File: omni_base_description/urdf/objects/antenna.urdf.xacro (robot description, xacro)
@@ -25,5 +25,10 @@
         <origin xyz="0 0 0" rpy="0 0 0" />
         <geometry>
-          <mesh filename="package://omni_base_description/meshes/base/base_antena_link.stl" scale="1 ${reflect} 1" />
+          <xacro:if value="${reflect == 1}">
+            <mesh filename="package://omni_base_description/meshes/base/base_antenna_link.stl" scale="1 1 1" />
+          </xacro:if>
+          <xacro:unless value="${reflect == 1}">
+            <mesh filename="package://omni_base_description/meshes/base/base_antenna_link_mirror.stl" scale="1 1 1"/>
+          </xacro:unless>
         </geometry>
         <material name="">
@@ -34,5 +39,10 @@
         <origin xyz="0 0 0" rpy="0 0 0" />
         <geometry>
-          <mesh filename="package://omni_base_description/meshes/base/base_antena_link.stl" scale="1 ${reflect} 1"/>
+          <xacro:if value="${reflect == 1}">
+            <mesh filename="package://omni_base_description/meshes/base/base_antenna_link.stl" scale="1 1 1" />
+          </xacro:if>
+          <xacro:unless value="${reflect == 1}">
+            <mesh filename="package://omni_base_description/meshes/base/base_antenna_link_mirror.stl" scale="1 1 1"/>
+          </xacro:unless>
         </geometry>
       </collision>

File: omni_base_description/urdf/wheels/wheel.gazebo.xacro (robot description, xacro)
@@ -1,2 +1,3 @@
+<?xml version="1.0"?>
 <!--
   Copyright (c) 2023 PAL Robotics S.L. All rights reserved.
@@ -11,19 +12,77 @@
   limitations under the License.
  -->
-<robot xmlns:xacro="http://ros.org/wiki/xacro">
+<robot xmlns:xacro="http://ros.org/wiki/xacro" xmlns:gz="http://gazebosim.org/schema">
   <!-- MACRO DEFINITION -->
   <xacro:macro name="wheel_gazebo" params="side">
     <!-- Contact model for the wheel surface -->
-    <gazebo reference="wheel_${side}_link">
-      <kp>1000000.0</kp>
-      <kd>1000.0</kd>
-      <mu1>0.0</mu1>
-      <mu2>0.0</mu2>
-      <fdir1>1 0 0</fdir1>
-      <maxVel>1.0</maxVel>
-      <minDepth>0.00</minDepth>
-      <implicitSpringDamper>1</implicitSpringDamper>
-      <material>Gazebo/Grey</material>
-    </gazebo>
+    <xacro:if value="${gazebo_version == 'classic'}">
+      <gazebo reference="wheel_${side}_link">
+        <kp>1000000.0</kp>
+        <kd>1000.0</kd>
+        <mu1>0.0</mu1>
+        <mu2>0.0</mu2>
+        <fdir1>1 0 0</fdir1>
+        <maxVel>1.0</maxVel>
+        <minDepth>0.00</minDepth>
+        <implicitSpringDamper>1</implicitSpringDamper>
+        <material>Gazebo/Grey</material>
+      </gazebo>
+    </xacro:if>
+    <xacro:if value="${gazebo_version == 'gazebo'}">
+      <gazebo reference="wheel_${side}_link">
+      <collision>
+          <surface>
+            <friction>
+              <ode>
+                <!-- <mu> : Coefficient of friction in first friction pyramid direction,
+                the unitless maximum ratio of force in first friction pyramid direction to normal force. -->
+                <!-- <mu2> : Coefficient of friction in second friction pyramid direction,
+                the unitless maximum ratio of force in second friction pyramid direction to normal force. -->
+                <!-- <fdir1> : Unit vector specifying first friction pyramid direction in
+                collision-fixed reference frame. If the friction pyramid model is in use, and this value
+                is set to a unit vector for one of the colliding surfaces, the ODE Collide callback
+                function will align the friction pyramid directions with a reference frame fixed to that
+                collision surface. If both surfaces have this value set to a vector of zeros, the friction
+                pyramid directions will be aligned with the world frame. If this value is set for both
+                surfaces, the behavior is undefined. -->
+                <!-- <slip1> : Force dependent slip in first friction pyramid direction,
+                equivalent to inverse of viscous damping coefficient with units of m/s/N.
+                A slip value of 0 is infinitely viscous. -->
+                <!-- <slip2> : Force dependent slip in second friction pyramid direction,
+                equivalent to inverse of viscous damping coefficient with units of m/s/N.
+                A slip value of 0 is infinitely viscous. -->
+                <mu>0.01</mu>
+                <mu2>0.0</mu2>
+                <xacro:if value="${side == 'front_left'}">
+                  <fdir1 gz:expressed_in="base_footprint">1 -1 0</fdir1>
+                </xacro:if>
+                <xacro:if value="${side == 'rear_left'}">
+                  <fdir1 gz:expressed_in="base_footprint">1 1 0</fdir1>
+                </xacro:if>
+                <xacro:if value="${side == 'front_right'}">
+                  <fdir1 gz:expressed_in="base_footprint">1 1 0</fdir1>
+                </xacro:if>
+                <xacro:if value="${side == 'rear_right'}">
+                  <fdir1 gz:expressed_in="base_footprint">1 -1 0</fdir1>
+                </xacro:if>
+              </ode>
+            </friction>
+            <contact>
+              <ode>
+                <!-- <kp> : dynamically "stiffness"-equivalent coefficient for contact joints. -->
+                <!-- <kd> : dynamically "damping"-equivalent coefficient for contact joints. -->
+                <!-- <max_vel> : maximum contact correction velocity truncation term. -->
+                <!-- <min_depth> : minimum allowable depth before contact correction impulse is applied. -->
+                <kp>10.0</kp>
+                <kd>10.0</kd>
+                <max_vel>1.0</max_vel>
+                <min_depth>0.0</min_depth>
+              </ode>
+            </contact>
+          </surface>
+        </collision>
+        <material>Gazebo/Grey</material>
+      </gazebo>
+    </xacro:if>
   </xacro:macro>
 </robot>

File: omni_base_description/urdf/wheels/wheel.urdf.xacro (robot description, xacro)
@@ -30,8 +30,8 @@
         <geometry>
           <xacro:if value="${frontal_reflect == 1}">
-            <mesh filename="package://omni_base_description/meshes/wheels/suspension_front_link.stl" scale="1 ${sagital_reflect} 1"/>
+            <mesh filename="package://omni_base_description/meshes/wheels/suspension_front_link.stl" scale="1 1 1"/>
           </xacro:if>
           <xacro:unless value="${frontal_reflect == 1}">
-            <mesh filename="package://omni_base_description/meshes/wheels/suspension_rear_link.stl" scale="1 ${sagital_reflect} 1"/>
+            <mesh filename="package://omni_base_description/meshes/wheels/suspension_rear_link.stl" scale="1 1 1"/>
           </xacro:unless>
         </geometry>
@@ -44,8 +44,8 @@
         <geometry>
           <xacro:if value="${frontal_reflect == 1}">
-            <mesh filename="package://omni_base_description/meshes/wheels/suspension_front_link.stl" scale="1 ${sagital_reflect} 1"/>
+            <mesh filename="package://omni_base_description/meshes/wheels/suspension_front_link.stl" scale="1 1 1"/>
           </xacro:if>
           <xacro:unless value="${frontal_reflect == 1}">
-            <mesh filename="package://omni_base_description/meshes/wheels/suspension_rear_link.stl" scale="1 ${sagital_reflect} 1"/>
+            <mesh filename="package://omni_base_description/meshes/wheels/suspension_rear_link.stl" scale="1 1 1"/>
           </xacro:unless>
         </geometry>
@@ -71,5 +71,10 @@
         <origin xyz="0 0 0" rpy="0 0 0" />
         <geometry>
-          <mesh filename="package://omni_base_description/meshes/wheels/wheel_link.stl" scale="1 1 ${sagital_reflect}"/>
+          <xacro:if value="${sagital_reflect == 1}">
+            <mesh filename="package://omni_base_description/meshes/wheels/wheel_link.stl" scale="1 1 1"/>
+          </xacro:if>
+          <xacro:unless value="${sagital_reflect == 1}">
+            <mesh filename="package://omni_base_description/meshes/wheels/wheel_link_reverted.stl" scale="1 1 1"/>
+          </xacro:unless>
         </geometry>
         <material name="DarkGrey"/>
