Commit message: update the information of the front-right and rear-left laser sensor

File: omni_base_description/robots/omni_base.urdf.xacro (robot description, xacro)
@@ -8,11 +8,16 @@
 -->
 <robot  xmlns:xacro="http://ros.org/wiki/xacro" name="omni_base" >
-  <xacro:arg name="laser_model" default="sick-571"/> <!-- false, hokuyo, sick-551, sick-561, sick-571-->
+  <xacro:arg name="front_right_laser_model" default="sick-571"/> <!-- false, hokuyo, sick-551, sick-561, sick-571-->
+  <xacro:arg name="rear_left_laser_model" default="sick-571"/> <!-- false, hokuyo, sick-551, sick-561, sick-571-->
   <xacro:arg name="multiple" default="false"/>
   <xacro:arg name="namespace" default=""/>
-  <xacro:property name="laser_model" value="$(arg laser_model)" />
+  <xacro:property name="front_right_laser_model" value="$(arg front_right_laser_model)" />
+  <xacro:property name="rear_left_laser_model" value="$(arg rear_left_laser_model)" />
   <xacro:property name="is_multiple" value="$(arg multiple)" />
   <xacro:property name="nsp" value="$(arg namespace)" />
-  <xacro:if value="${laser_model not in ['false', 'sick-551', 'sick-561', 'sick-571', 'hokuyo']}">
+  <xacro:if value="${front_right_laser_model not in ['false', 'sick-551', 'sick-561', 'sick-571', 'hokuyo']}">
+    <xacro:wrong_laser_model/>
+  </xacro:if>
+  <xacro:if value="${rear_left_laser_model not in ['false', 'sick-551', 'sick-561', 'sick-571', 'hokuyo']}">
     <xacro:wrong_laser_model/>
   </xacro:if>
@@ -25,4 +30,4 @@
   <xacro:include filename="$(find omni_base_description)/urdf/materials.urdf.xacro" />
   <!-- Now we can start using the macros included above to define the actual robot -->
-  <xacro:base_sensors name="base" laser_model="$(arg laser_model)"/>
+  <xacro:base_sensors name="base" front_right_laser_model="$(arg front_right_laser_model)" rear_left_laser_model="$(arg rear_left_laser_model)"/>
 </robot>

File: omni_base_description/urdf/base/base_sensors.urdf.xacro (robot description, xacro)
@@ -9,7 +9,39 @@
 <robot xmlns:xacro="http://ros.org/wiki/xacro">
   <xacro:include filename="$(find omni_base_description)/urdf/base/base.urdf.xacro"/>
+  <xacro:include filename="$(find pmb2_description)/urdf/sensors/hokuyo_urg_04lx_ug01_laser.urdf.xacro"/>
+  <xacro:include filename="$(find pmb2_description)/urdf/sensors/sick_tim551_laser.urdf.xacro"/>
   <xacro:include filename="$(find pmb2_description)/urdf/sensors/sick_tim561_laser.urdf.xacro"/>
-  <!-- laser_model can be: false, hokuyo, sick-551, sick-561, sick-571-->
-  <xacro:macro name="base_sensors" params=" name laser_model:=sick-571">
+  <xacro:include filename="$(find pmb2_description)/urdf/sensors/sick_tim571_laser.urdf.xacro"/>
+  <!-- Laser model can be: false, hokuyo, sick-551, sick-561, sick-571-->
+  <!-- Laser:  Theoretic FOV = 220 -->
+  <xacro:macro name="laser_sensor" params="name parent model ros_topic *origin update_rate:=10 min_angle:=${-110 * deg_to_rad} max_angle:=${110 * deg_to_rad}">
+    <xacro:if value="${model == 'sick-551'}">
+      <!-- Rear Laser:  Theoretic FOV = 220 -->
+      <xacro:sick_tim551_laser name="${name}" parent="${parent}" ros_topic="${ros_topic}" update_rate="${update_rate}" min_angle="${min_angle}" max_angle="${max_angle}" >
+        <xacro:insert_block name="origin" />
+      </xacro:sick_tim551_laser>
+    </xacro:if>
+    <xacro:if value="${model == 'sick-561'}">
+      <!-- Rear Laser:  Theoretic FOV = 220 -->
+      <xacro:sick_tim561_laser name="${name}" parent="${parent}" ros_topic="${ros_topic}" update_rate="${update_rate}" min_angle="${min_angle}" max_angle="${max_angle}" >
+        <xacro:insert_block name="origin" />
+      </xacro:sick_tim561_laser>
+    </xacro:if>
+    <xacro:if value="${model == 'sick-571'}">
+      <!-- Rear Laser:  Theoretic FOV = 220 -->
+      <xacro:sick_tim571_laser name="${name}" parent="${parent}" ros_topic="${ros_topic}" update_rate="${update_rate}" min_angle="${min_angle}" max_angle="${max_angle}" >
+        <xacro:insert_block name="origin" />
+      </xacro:sick_tim571_laser>
+    </xacro:if>
+    <xacro:if value="${model == 'hokuyo'}">
+      <!-- Rear Laser:  Theoretic FOV = 220 -->
+      <xacro:hokuyo_urg_041x_ug01_laser name="${name}" parent="${parent}" ros_topic="${ros_topic}" update_rate="${update_rate}" min_angle="${min_angle}" max_angle="${max_angle}" >
+        <xacro:insert_block name="origin" />
+      </xacro:hokuyo_urg_041x_ug01_laser>
+    </xacro:if>
+  </xacro:macro>
+  <!-- front_right_laser_model can be: false, hokuyo, sick-551, sick-561, sick-571-->
+  <!-- rear_left_laser_model can be: false, hokuyo, sick-551, sick-561, sick-571-->
+  <xacro:macro name="base_sensors" params=" name front_right_laser_model:=sick-571 rear_left_laser_model:=sick-571">
     <!-- Base Laser Link -->
     <joint name="${name}_laser_joint" type="fixed">
@@ -25,11 +57,12 @@
         </inertial>
     </link>
-    <!-- Rear Laser:  Theoretic FOV = 220 -->
-    <xacro:sick_tim561_laser name="${name}_rear_laser" parent="${name}" ros_topic="scan_rear_raw" update_rate="10" min_angle="${-120 * deg_to_rad}" max_angle="${120 * deg_to_rad}"  >
-      <origin xyz="-0.277 0 0.15614" rpy="0 0 ${180 * deg_to_rad}" />
-    </xacro:sick_tim561_laser>
-    <xacro:sick_tim561_laser name="${name}_front_laser" parent="${name}" ros_topic="scan_front_raw" update_rate="10" min_angle="${-120 * deg_to_rad}" max_angle="${120 * deg_to_rad}" >
-      <origin xyz="0.277 0 0.15614" rpy="0 0 0" />
-    </xacro:sick_tim561_laser>
+    <!-- Rear Laser Sensor -->
+    <xacro:laser_sensor name="${name}_rear_laser" parent="${name}" model="${rear_left_laser_model}" ros_topic="scan_rear_raw">
+      <origin xyz="-0.27512 0.18297 0.13244" rpy="${-180 * deg_to_rad} 0 ${135 * deg_to_rad}" />
+    </xacro:laser_sensor>
+    <!-- Front Laser Sensor -->
+    <xacro:laser_sensor name="${name}_front_laser" parent="${name}" model="${front_right_laser_model}" ros_topic="scan_rear_raw">
+    <origin xyz="0.27512 -0.18297 0.13244" rpy="${-180 * deg_to_rad} 0 ${-45 * deg_to_rad}" />
+    </xacro:laser_sensor>
     <xacro:base name="${name}"/>
   </xacro:macro>

Commit message: fix the laser model naming for front and rear sensors

File: omni_base_description/robots/omni_base.urdf.xacro (robot description, xacro)
@@ -8,16 +8,16 @@
 -->
 <robot  xmlns:xacro="http://ros.org/wiki/xacro" name="omni_base" >
-  <xacro:arg name="front_right_laser_model" default="sick-571"/> <!-- false, hokuyo, sick-551, sick-561, sick-571-->
-  <xacro:arg name="rear_left_laser_model" default="sick-571"/> <!-- false, hokuyo, sick-551, sick-561, sick-571-->
+  <xacro:arg name="front_laser_model" default="sick-571"/> <!-- false, hokuyo, sick-551, sick-561, sick-571-->
+  <xacro:arg name="rear_laser_model" default="sick-571"/> <!-- false, hokuyo, sick-551, sick-561, sick-571-->
   <xacro:arg name="multiple" default="false"/>
   <xacro:arg name="namespace" default=""/>
-  <xacro:property name="front_right_laser_model" value="$(arg front_right_laser_model)" />
-  <xacro:property name="rear_left_laser_model" value="$(arg rear_left_laser_model)" />
+  <xacro:property name="front_laser_model" value="$(arg front_laser_model)" />
+  <xacro:property name="rear_laser_model" value="$(arg rear_laser_model)" />
   <xacro:property name="is_multiple" value="$(arg multiple)" />
   <xacro:property name="nsp" value="$(arg namespace)" />
-  <xacro:if value="${front_right_laser_model not in ['false', 'sick-551', 'sick-561', 'sick-571', 'hokuyo']}">
+  <xacro:if value="${front_laser_model not in ['false', 'sick-551', 'sick-561', 'sick-571', 'hokuyo']}">
     <xacro:wrong_laser_model/>
   </xacro:if>
-  <xacro:if value="${rear_left_laser_model not in ['false', 'sick-551', 'sick-561', 'sick-571', 'hokuyo']}">
+  <xacro:if value="${rear_laser_model not in ['false', 'sick-551', 'sick-561', 'sick-571', 'hokuyo']}">
     <xacro:wrong_laser_model/>
   </xacro:if>
@@ -30,4 +30,4 @@
   <xacro:include filename="$(find omni_base_description)/urdf/materials.urdf.xacro" />
   <!-- Now we can start using the macros included above to define the actual robot -->
-  <xacro:base_sensors name="base" front_right_laser_model="$(arg front_right_laser_model)" rear_left_laser_model="$(arg rear_left_laser_model)"/>
+  <xacro:base_sensors name="base" front_laser_model="$(arg front_laser_model)" rear_laser_model="$(arg rear_laser_model)"/>
 </robot>

File: omni_base_description/urdf/base/base_sensors.urdf.xacro (robot description, xacro)
@@ -42,13 +42,13 @@
     </xacro:if>
   </xacro:macro>
-  <!-- front_right_laser_model can be: false, hokuyo, sick-551, sick-561, sick-571-->
-  <!-- rear_left_laser_model can be: false, hokuyo, sick-551, sick-561, sick-571-->
-  <xacro:macro name="base_sensors" params=" name front_right_laser_model:=sick-571 rear_left_laser_model:=sick-571">
+  <!-- front_laser_model can be: false, hokuyo, sick-551, sick-561, sick-571-->
+  <!-- rear_laser_model can be: false, hokuyo, sick-551, sick-561, sick-571-->
+  <xacro:macro name="base_sensors" params=" name front_laser_model:=sick-571 rear_laser_model:=sick-571">
   <!-- Rear Laser Sensor -->
-  <xacro:laser_sensor name="${name}_rear_laser" parent="${name}" model="${rear_left_laser_model}" ros_topic="scan_rear_raw">
+  <xacro:laser_sensor name="${name}_rear_laser" parent="${name}" model="${rear_laser_model}" ros_topic="scan_rear_raw">
     <origin xyz="-0.27512 0.18297 0.13244" rpy="${-180 * deg_to_rad} 0 ${135 * deg_to_rad}" />
   </xacro:laser_sensor>
   <!-- Front Laser Sensor -->
-  <xacro:laser_sensor name="${name}_front_laser" parent="${name}" model="${front_right_laser_model}" ros_topic="scan_rear_raw">
+  <xacro:laser_sensor name="${name}_front_laser" parent="${name}" model="${front_laser_model}" ros_topic="scan_front_raw">
   <origin xyz="0.27512 -0.18297 0.13244" rpy="${-180 * deg_to_rad} 0 ${-45 * deg_to_rad}" />
   </xacro:laser_sensor>

Commit message: Use urdf_utils

File: omni_base_description/robots/omni_base.urdf.xacro (robot description, xacro)
@@ -23,4 +23,6 @@
   </xacro:if>
   <!-- The following included files set up definitions of parts of the robot body -->
+  <!--File includes-->
+  <xacro:include filename="$(find pal_urdf_utils)/urdf/deg_to_rad.xacro" />
   <!-- Base -->
   <xacro:include filename="$(find omni_base_description)/urdf/base/base_sensors.urdf.xacro" />
@@ -28,5 +30,5 @@
   <xacro:include filename="$(find omni_base_description)/gazebo/gazebo.urdf.xacro" />
   <!-- Materials for visualization -->
-  <xacro:include filename="$(find omni_base_description)/urdf/materials.urdf.xacro" />
+  <xacro:include filename="$(find pal_urdf_utils)/urdf/materials.urdf.xacro" />
   <!-- Now we can start using the macros included above to define the actual robot -->
   <xacro:base_sensors name="base" front_laser_model="$(arg front_laser_model)" rear_laser_model="$(arg rear_laser_model)"/>

File: omni_base_description/urdf/base/antenna.urdf.xacro (robot description, xacro)
@@ -26,7 +26,5 @@
           <mesh filename="package://omni_base_description/meshes/base/base_antena_link.stl" scale="1 ${reflect} 1" />
         </geometry>
-        <material name="">
-          <color rgba="0.75294 0.75294 0.75294 1" />
-        </material>
+        <material name="FlatBlack" />
       </visual>
       <collision>

File: omni_base_description/urdf/base/base.urdf.xacro (robot description, xacro)
@@ -8,5 +8,4 @@
 -->
 <robot xmlns:xacro="http://ros.org/wiki/xacro">
-  <xacro:include filename="$(find omni_base_description)/urdf/deg_to_rad.xacro"/>
   <xacro:include filename="$(find omni_base_description)/urdf/wheels/wheel.urdf.xacro"/>
   <xacro:include filename="$(find omni_base_description)/urdf/base/antenna.urdf.xacro"/>
@@ -34,7 +33,5 @@
           <mesh filename="package://omni_base_description/meshes/base/base_link.stl" />
         </geometry>
-        <material name="">
-          <color rgba="0.75294 0.75294 0.75294 1" />
-        </material>
+        <material name="White" />
       </visual>
       <collision>
@@ -91,7 +88,5 @@
           <mesh filename="package://omni_base_description/meshes/base/base_dock_link.stl" />
         </geometry>
-        <material name="">
-          <color rgba="0.25098 0.25098 0.25098 1" />
-        </material>
+        <material name="FlatBlack" />
       </visual>
       <collision>
@@ -102,4 +97,7 @@
       </collision>
     </link>
+    <gazebo reference="${name}_dock_link">
+      <material>Gazebo/Black</material>
+    </gazebo>
     <joint name="${name}_dock" type="fixed">
       <origin xyz="0.3535 0 0.0596" rpy="0 0 0" />

File: omni_base_description/urdf/base/base_sensors.urdf.xacro (robot description, xacro)
@@ -13,5 +13,4 @@
   <xacro:include filename="$(find pmb2_description)/urdf/sensors/sick_tim561_laser.urdf.xacro"/>
   <xacro:include filename="$(find pmb2_description)/urdf/sensors/sick_tim571_laser.urdf.xacro"/>
-  <xacro:include filename="$(find omni_base_description)/urdf/deg_to_rad.xacro"/>
   <!-- Laser model can be: false, hokuyo, sick-551, sick-561, sick-571-->
   <xacro:macro name="laser_sensor" params="name parent model ros_topic *origin update_rate:=10">

File: omni_base_description/urdf/wheels/wheel.gazebo.xacro (robot description, xacro)
@@ -19,5 +19,5 @@
       <minDepth>0.00</minDepth>
       <implicitSpringDamper>1</implicitSpringDamper>
-      <material>Gazebo/DarkGrey</material>
+      <material>Gazebo/Grey</material>
     </gazebo>
   </xacro:macro>

File: omni_base_description/urdf/wheels/wheel.urdf.xacro (robot description, xacro)
@@ -68,5 +68,5 @@
           <mesh filename="package://omni_base_description/meshes/wheels/wheel_link.stl" scale="1 1 ${sagital_reflect}"/>
         </geometry>
-        <material name="DarkGrey"/>
+        <material name="Grey"/>
       </visual>
       <collision>

Commit message: fix lidar mesh issues and using light base stl

File: omni_base_description/robots/omni_base.urdf.xacro (robot description, xacro)
@@ -14,6 +14,6 @@
 <robot  xmlns:xacro="http://ros.org/wiki/xacro" name="omni_base" >
   <xacro:arg name="use_sim" default="true"/>
-  <xacro:arg name="front_laser_model" default="sick-561"/> <!-- false, hokuyo, sick-551, sick-561, sick-571-->
-  <xacro:arg name="rear_laser_model" default="sick-561"/> <!-- false, hokuyo, sick-551, sick-561, sick-571-->
+  <xacro:arg name="front_laser_model" default="sick-571"/> <!-- false, hokuyo, sick-551, sick-561, sick-571-->
+  <xacro:arg name="rear_laser_model" default="sick-571"/> <!-- false, hokuyo, sick-551, sick-561, sick-571-->
   <xacro:arg name="multiple" default="false"/>
   <xacro:arg name="namespace" default=""/>

File: omni_base_description/urdf/base/base_sensors.urdf.xacro (robot description, xacro)
@@ -9,5 +9,8 @@
 <robot xmlns:xacro="http://ros.org/wiki/xacro">
   <xacro:include filename="$(find omni_base_description)/urdf/base/base.urdf.xacro"/>
+  <xacro:include filename="$(find omni_base_description)/urdf/sensors/hokuyo_urg_04lx_ug01_laser.urdf.xacro"/>
+  <xacro:include filename="$(find omni_base_description)/urdf/sensors/sick_tim551_laser.urdf.xacro"/>
   <xacro:include filename="$(find omni_base_description)/urdf/sensors/sick_tim561_laser.urdf.xacro"/>
+  <xacro:include filename="$(find omni_base_description)/urdf/sensors/sick_tim571_laser.urdf.xacro"/>
   <xacro:include filename="$(find omni_base_description)/urdf/deg_to_rad.xacro"/>
   <!-- Laser model can be: false, hokuyo, sick-551, sick-561, sick-571-->

File: omni_base_description/urdf/sensors/hokuyo_urg_04lx_ug01_laser.urdf.xacro (robot description, xacro)
@@ -13,18 +13,18 @@
  -->
 <robot xmlns:xacro="http://ros.org/wiki/xacro">
-  <xacro:include filename="$(find omni_base_description)/urdf/sensors/sick_tim561_laser.gazebo.xacro" />
-  <xacro:macro name="sick_tim561_laser" params="name parent *origin ros_topic update_rate min_angle max_angle">
-     <link name="${name}_link" type="laser">
+  <xacro:include filename="$(find omni_base_description)/urdf/sensors/hokuyo_urg_04lx_ug01_laser.gazebo.xacro" />
+  <xacro:macro name="hokuyo_urg_04lx_ug01_laser" params="name parent *origin ros_topic update_rate min_angle max_angle">
+    <link name="${name}_link" type="laser">
       <inertial>
-        <origin xyz="-0.02559000000 -0.00056000000 -0.05732000000" rpy="0 0 0"/>
-        <mass value="0.28922000000"/>
-        <inertia ixx="0.00002628919" ixy="0.00000024298" ixz="-0.00000368129"
-                 iyy="0.00003374542" iyz="-0.00000001330"
-                 izz="0.00005832599"/>
+        <origin xyz="0 0 -0.04480000000" rpy="0 0 0"/>
+        <mass value="0.22963000000"/>
+        <inertia ixx="0.00003393164" ixy="0.00000064943" ixz="0.00000000000"
+                 iyy="0.00001849658" iyz="0.00000000000"
+                 izz="0.00005027615"/>
       </inertial>
       <visual>
         <origin xyz="0 0 0" rpy="0 0 0" />
         <geometry>
-          <mesh filename="package://omni_base_description/meshes/sensors/sick_tim551.stl" scale="1 1 1"/>
+          <mesh filename="package://omni_base_description/meshes/sensors/hokuyo_urg_04lx_ug01.stl"/>
         </geometry>
         <material name="DarkGrey"/>
@@ -44,5 +44,5 @@
     </joint>
     <!-- gazebo extensions -->
-    <xacro:sick_tim561_laser_gazebo name="${name}" ros_topic="${ros_topic}" update_rate="${update_rate}" min_angle="${min_angle}" max_angle="${max_angle}" />
+    <xacro:hokuyo_urg_04lx_ug01_laser_gazebo name="${name}" ros_topic="${ros_topic}" update_rate="${update_rate}" min_angle="${min_angle}" max_angle="${max_angle}" />
   </xacro:macro>
 </robot>

File: omni_base_description/urdf/sensors/sick_tim551_laser.urdf.xacro (robot description, xacro)
@@ -13,6 +13,6 @@
  -->
 <robot xmlns:xacro="http://ros.org/wiki/xacro">
-  <xacro:include filename="$(find omni_base_description)/urdf/sensors/sick_tim561_laser.gazebo.xacro" />
-  <xacro:macro name="sick_tim561_laser" params="name parent *origin ros_topic update_rate min_angle max_angle">
+  <xacro:include filename="$(find omni_base_description)/urdf/sensors/sick_tim551_laser.gazebo.xacro" />
+  <xacro:macro name="sick_tim551_laser" params="name parent *origin ros_topic update_rate min_angle max_angle">
      <link name="${name}_link" type="laser">
       <inertial>
@@ -44,5 +44,5 @@
     </joint>
     <!-- gazebo extensions -->
-    <xacro:sick_tim561_laser_gazebo name="${name}" ros_topic="${ros_topic}" update_rate="${update_rate}" min_angle="${min_angle}" max_angle="${max_angle}" />
+    <xacro:sick_tim551_laser_gazebo name="${name}" ros_topic="${ros_topic}" update_rate="${update_rate}" min_angle="${min_angle}" max_angle="${max_angle}" />
   </xacro:macro>
 </robot>

File: omni_base_description/urdf/sensors/sick_tim571_laser.urdf.xacro (robot description, xacro)
@@ -13,6 +13,6 @@
  -->
 <robot xmlns:xacro="http://ros.org/wiki/xacro">
-  <xacro:include filename="$(find omni_base_description)/urdf/sensors/sick_tim561_laser.gazebo.xacro" />
-  <xacro:macro name="sick_tim561_laser" params="name parent *origin ros_topic update_rate min_angle max_angle">
+  <xacro:include filename="$(find omni_base_description)/urdf/sensors/sick_tim571_laser.gazebo.xacro" />
+  <xacro:macro name="sick_tim571_laser" params="name parent *origin ros_topic update_rate min_angle max_angle">
      <link name="${name}_link" type="laser">
       <inertial>
@@ -44,5 +44,5 @@
     </joint>
     <!-- gazebo extensions -->
-    <xacro:sick_tim561_laser_gazebo name="${name}" ros_topic="${ros_topic}" update_rate="${update_rate}" min_angle="${min_angle}" max_angle="${max_angle}" />
+    <xacro:sick_tim571_laser_gazebo name="${name}" ros_topic="${ros_topic}" update_rate="${update_rate}" min_angle="${min_angle}" max_angle="${max_angle}" />
   </xacro:macro>
 </robot>

Commit message: Set use_sim_time false as default

File: omni_base_description/robots/omni_base.urdf.xacro (robot description, xacro)
@@ -13,5 +13,5 @@
  -->
 <robot  xmlns:xacro="http://ros.org/wiki/xacro" name="omni_base" >
-  <xacro:arg name="use_sim" default="true"/>
+  <xacro:arg name="use_sim" default="false"/>
   <xacro:arg name="front_laser_model" default="sick-571"/> <!-- false, hokuyo, sick-551, sick-561, sick-571-->
   <xacro:arg name="rear_laser_model" default="sick-571"/> <!-- false, hokuyo, sick-551, sick-561, sick-571-->

File: omni_base_description/ros2_control/ros2_control.urdf.xacro (robot description, xacro)
@@ -14,5 +14,5 @@
 <robot xmlns:xacro="http://ros.org/wiki/xacro"
        name="omni_base" >
-<xacro:macro name="omni_base_ros2_control" params="use_sim:=^|true">
+<xacro:macro name="omni_base_ros2_control" params="use_sim:=^|false">
     <xacro:include filename="$(find omni_base_description)/urdf/wheels/wheel.ros2_control.xacro"/>
     <xacro:include filename="$(find omni_base_description)/urdf/sensors/sensors.ros2_control.xacro"/>

Commit message: init support to namespaces

File: omni_base_description/robots/omni_base.urdf.xacro (robot description, xacro)
@@ -24,5 +24,4 @@
   <!-- Execution env config -->
   <xacro:arg name="use_sim_time" default="false"/>
-  <xacro:arg name="is_multiple" default="false"/>
   <xacro:arg name="namespace" default=""/>
   <xacro:arg name="is_public_sim" default="false"/>
@@ -48,5 +47,4 @@
   <!-- Execution env configuration -->
   <xacro:property name="use_sim_time" default="$(arg use_sim_time)"/>
-  <xacro:property name="is_multiple" value="$(arg is_multiple)" />
   <xacro:property name="namespace" value="$(arg namespace)" />
   <xacro:property name="is_public_sim" value="$(arg is_public_sim)" />

File: omni_base_description/ros2_control/ros2_control.urdf.xacro (robot description, xacro)
@@ -20,5 +20,10 @@
     <xacro:if value="${use_sim_time}">
       <gazebo>
-        <plugin filename="libgazebo_ros2_control.so" name="gazebo_ros2_control">
+        <plugin filename="libgazebo_ros2_control.so" name="${namespace}gazebo_ros2_control">
+          <ros>
+            <namespace>/${namespace}</namespace>
+            <remapping>/tf:=${namespace}/tf</remapping>
+          </ros>
+          <robot_param_node>${namespace}/robot_state_publisher</robot_param_node>
           <parameters>$(find omni_base_description)/ros2_control/gazebo_controller_manager_cfg.yaml</parameters>
           <!-- <robot_sim_type>gazebo_ros2_control/GazeboSystem</robot_sim_type>

File: omni_base_description/urdf/base/base.gazebo.xacro (robot description, xacro)
@@ -34,4 +34,5 @@
       <plugin name="gazebo_ros_planar_move" filename="libgazebo_ros_planar_move.so">
         <ros>
+          <namespace>/${namespace}</namespace>
           <remapping>cmd_vel:=mobile_base_controller/cmd_vel_unstamped</remapping>
           <remapping>odom:=mobile_base_controller/odom</remapping>
@@ -46,7 +47,4 @@
           <publish_odom_tf>false</publish_odom_tf>
         </xacro:unless>
-          <xacro:if value="${is_multiple}">
-            <namespace>/${nsp}</namespace>
-          </xacro:if>
         <odometry_frame>odom</odometry_frame>
         <robot_base_frame>base_footprint</robot_base_frame>
