Commit message: changed name from camera_on_top to camera_horizon_add_on

File: omni_base_description/robots/omni_base.urdf.xacro (robot description, xacro)
@@ -40,5 +40,5 @@
     <xacro:wrong_laser_model/>
   </xacro:if>
-  <xacro:if value="${add_on_module not in ['no-add-on', 'cobra', 'single']}">
+  <xacro:if value="${add_on_module not in ['no-add-on', 'cobra', 'horizon']}">
     <xacro:wrong_add_on_module/>
   </xacro:if>
@@ -59,10 +59,10 @@
     <xacro:cameras_add_on name="cameras_add_on" parent="base_link"/>
   </xacro:if>
-  <xacro:if value="${add_on_module == 'single'}">
-    <xacro:include filename="$(find omni_base_description)/urdf/cameras_add_on/camera_on_top.urdf.xacro" />
-    <xacro:camera_on_top name="camera_on_top" parent="base_link"/>
+  <xacro:if value="${add_on_module == 'horizon'}">
+    <xacro:include filename="$(find omni_base_description)/urdf/cameras_add_on/camera_horizon_add_on.urdf.xacro" />
+    <xacro:camera_horizon_add_on name="camera_horizon" parent="base_link"/>
   </xacro:if>
   <!-- Materials for visualization -->
-  <xacro:include filename="$(find pal_urdf_utils)/urdf/materials.urdf.xacro" />
+  <xacro:include filename="$(find pal_urdf_utils  )/urdf/materials.urdf.xacro" />
   <!-- Utils for degree to radian conversion -->
   <xacro:include filename="$(find pal_urdf_utils)/urdf/deg_to_rad.urdf.xacro" />

File: omni_base_description/urdf/cameras_add_on/camera_horizon_add_on.urdf.xacro (robot description, xacro)
@@ -13,6 +13,11 @@
 -->
 <robot xmlns:xacro="http://ros.org/wiki/xacro">
+  <xacro:include filename="$(find pal_urdf_utils)/urdf/deg_to_rad.urdf.xacro" />
+  <xacro:property name="use_sim_time" value="$(arg use_sim_time)" />
+  <xacro:property name="rgbd_x" value="0.28595"/>
+  <xacro:property name="rgbd_y" value="0.0"/>
+  <xacro:property name="rgbd_z" value="0.28125"/>
   <!-- MACRO DEFINITION -->
-  <xacro:macro name="camera_on_top" params="name parent">
+  <xacro:macro name="camera_horizon_add_on" params="name parent">
     <link name="${name}_link">
       <inertial>
@@ -26,5 +31,5 @@
           <origin xyz="0 0 0" rpy="0 0 0"/>
           <geometry>
-            <mesh filename="package://omni_base_description/meshes/cameras_add_on/camera_on_top.stl" scale="1 1 1"/>
+            <mesh filename="package://omni_base_description/meshes/cameras_add_on/camera_horizon.stl" scale="1 1 1"/>
           </geometry>
           <material name="White" />
@@ -33,5 +38,5 @@
           <origin xyz="0 0 0" rpy="0 0 0"/>
           <geometry>
-            <mesh filename="package://omni_base_description/meshes/cameras_add_on/camera_on_top.stl" scale="1 1 1"/>
+            <mesh filename="package://omni_base_description/meshes/cameras_add_on/camera_horizon.stl" scale="1 1 1"/>
           </geometry>
           <material name="White" />
@@ -45,4 +50,27 @@
       </joint>
     </xacro:macro>
-    <xacro:include filename="$(find omni_base_description)/urdf/sensors/camera_on_top.urdf.xacro" />
+    <xacro:if value="${camera_model == 'realsense-d435'}">
+      <xacro:include filename="$(find realsense2_description)/urdf/_d435.urdf.xacro" />
+      <xacro:sensor_d435
+        name="rgbd_camera"
+        parent="base_link"
+        topics_ns="rgbd_camera"
+        use_nominal_extrinsics="${use_sim_time}">
+        <origin
+            xyz="${rgbd_x} ${rgbd_y} ${rgbd_z}"
+            rpy="0.0 0.0 0.0"/>
+      </xacro:sensor_d435>
+    </xacro:if>
+    <xacro:if value="${camera_model == 'realsense-d435i'}">
+      <xacro:include filename="$(find realsense2_description)/urdf/_d435i.urdf.xacro" />
+      <xacro:sensor_d435i
+        name="rgbd_camera"
+        parent="base_link"
+        topics_ns="rgbd_camera"
+        use_nominal_extrinsics="${use_sim_time}">
+        <origin
+            xyz="${rgbd_x} ${rgbd_y} ${rgbd_z}"
+            rpy="0.0 0.0 0.0"/>
+      </xacro:sensor_d435i>
+    </xacro:if>
   </robot>

Commit message: Add gazebo_version xacro argument

File: omni_base_description/robots/omni_base.urdf.xacro (robot description, xacro)
@@ -26,4 +26,5 @@
   <xacro:arg name="namespace" default=""/>
   <xacro:arg name="is_public_sim" default="false"/>
+  <xacro:arg name="gazebo_version" default="classic"/>
   <!-- PROPERTIES -->
   <!-- HW configuration -->
@@ -49,4 +50,5 @@
   <xacro:property name="namespace" value="$(arg namespace)" />
   <xacro:property name="is_public_sim" value="$(arg is_public_sim)" />
+  <xacro:property name="gazebo_version" value="$(arg gazebo_version)"/>
   <!-- INCLUDES -->
   <!-- Base -->

Commit message: Support Mujoco

File: omni_base_description/robots/omni_base.urdf.xacro (robot description, xacro)
@@ -27,4 +27,9 @@
   <xacro:arg name="is_public_sim" default="false"/>
   <xacro:arg name="gazebo_version" default="classic"/>
+  <!-- mujoco-ros2-control, mujoco, gazebo, no-simulation -->
+  <xacro:arg name="sim_type" default="gazebo" />
+  <!-- false, position, motor -->
+  <xacro:arg name="mj_control" default="false" />
+  <xacro:arg name="world_name" default="floor" />
   <!-- PROPERTIES -->
   <!-- HW configuration -->
@@ -33,4 +38,15 @@
   <xacro:property name="add_on_module" value="$(arg add_on_module)"/>
   <xacro:property name="camera_model" value="$(arg camera_model)" />
+  <!-- Mujoco properties -->
+  <xacro:property name="sim_type" value="$(arg sim_type)" />
+  <xacro:property name="mj_control" value="$(arg mj_control)"/>
+  <xacro:property name="world_name" value="$(arg world_name)"/>
+  <!-- Properties check -->
+  <xacro:if value="${sim_type not in ['mujoco-ros2-control', 'mujoco', 'gazebo']}">
+    <xacro:wrong_sim_type />
+  </xacro:if>
+  <xacro:unless value="$(arg use_sim_time)">
+    <xacro:property name="sim_type" value="gazebo" />
+  </xacro:unless>
   <!-- HW configuration check -->
   <xacro:if value="${front_laser_model not in ['no-laser', 'sick-551', 'sick-561', 'sick-571', 'hokuyo']}">
@@ -68,8 +84,13 @@
   <xacro:include filename="$(find pal_urdf_utils)/urdf/deg_to_rad.urdf.xacro" />
   <!-- ROS 2 Control -->
-  <xacro:include filename="$(find omni_base_description)/ros2_control/ros2_control.urdf.xacro" />
-  <xacro:omni_base_ros2_control />
+  <xacro:if value="${sim_type != 'mujoco'}">
+    <xacro:include filename="$(find omni_base_description)/ros2_control/ros2_control.urdf.xacro" />
+    <xacro:omni_base_ros2_control sim_type="${sim_type}"/>
+  </xacro:if>
   <!-- ROBOT DEFINITION -->
   <!-- Now we can start using the macros included above to define the actual robot -->
   <xacro:base_sensors name="base" front_laser_model="$(arg front_laser_model)" rear_laser_model="$(arg rear_laser_model)"/>
+  <xacro:if value="${sim_type == 'mujoco' or sim_type == 'mujoco-ros2-control'}">
+    <xacro:base_mj world_name="${world_name}" mj_control="${mj_control}"/>
+  </xacro:if>
 </robot>

File: omni_base_description/ros2_control/ros2_control.urdf.xacro (robot description, xacro)
@@ -16,24 +16,26 @@
   <xacro:include filename="$(find omni_base_description)/urdf/wheels/wheel.ros2_control.xacro"/>
   <!-- MACRO DEFINITION-->
-  <xacro:macro name="omni_base_ros2_control">
+  <xacro:macro name="omni_base_ros2_control" params="use_sim_time:=^|false sim_type:=^|gazebo">
     <!-- Init the ROS 2 control gazebo interface -->
     <xacro:if value="${use_sim_time}">
-      <gazebo>
-        <xacro:if value="${gazebo_version == 'classic'}">
-          <plugin filename="libgazebo_ros2_control.so" name="gazebo_ros2_control">
-            <ros>
-              <namespace>${namespace}</namespace>
-              <remapping>/tf:=tf</remapping>
-              <remapping>/tf_static:=tf_static</remapping>
-            </ros>
-            <parameters>$(find omni_base_description)/ros2_control/gazebo_controller_manager_cfg.yaml</parameters>
-          </plugin>
-        </xacro:if>
-        <xacro:if value="${gazebo_version == 'gazebo'}">
-          <plugin filename="gz_ros2_control-system" name="gz_ros2_control::GazeboSimROS2ControlPlugin">
-            <parameters>$(find omni_base_description)/ros2_control/gazebo_controller_manager_cfg.yaml</parameters>
-          </plugin>
-        </xacro:if>
-      </gazebo>
+      <xacro:if value="${sim_type == 'gazebo'}">
+        <gazebo>
+          <xacro:if value="${gazebo_version == 'classic'}">
+            <plugin filename="libgazebo_ros2_control.so" name="gazebo_ros2_control">
+              <ros>
+                <namespace>${namespace}</namespace>
+                <remapping>/tf:=tf</remapping>
+                <remapping>/tf_static:=tf_static</remapping>
+              </ros>
+              <parameters>$(find omni_base_description)/ros2_control/gazebo_controller_manager_cfg.yaml</parameters>
+            </plugin>
+          </xacro:if>
+          <xacro:if value="${gazebo_version == 'gazebo'}">
+            <plugin filename="gz_ros2_control-system" name="gz_ros2_control::GazeboSimROS2ControlPlugin">
+              <parameters>$(find omni_base_description)/ros2_control/gazebo_controller_manager_cfg.yaml</parameters>
+            </plugin>
+          </xacro:if>
+        </gazebo>
+      </xacro:if>
     </xacro:if>
     <!-- ROS 2 control config-->
@@ -43,9 +45,17 @@
         <!-- HW interface; gazebo-->
         <hardware>
-          <xacro:if value="${gazebo_version == 'classic'}">
-            <plugin>gazebo_ros2_control/GazeboSystem</plugin>
+          <xacro:if value="${sim_type == 'mujoco-ros2-control'}">
+            <plugin>mujoco_ros2_control/MujocoSystemInterface</plugin>
+            <!-- Override the slowdown settings in the Simulate App and run at 3x speed -->
+            <param name="sim_speed_factor">1.0</param>
+            <!-- <param name="pids_config_file">$(find omni_base_mujoco)/config/pids.yaml</param> -->
           </xacro:if>
-          <xacro:if value="${gazebo_version == 'gazebo'}">
-            <plugin>gz_ros2_control/GazeboSimSystem</plugin>
+          <xacro:if value="${sim_type == 'gazebo'}">
+            <xacro:if value="${gazebo_version == 'classic'}">
+              <plugin>gazebo_ros2_control/GazeboSystem</plugin>
+            </xacro:if>
+            <xacro:if value="${gazebo_version == 'gazebo'}">
+              <plugin>gz_ros2_control/GazeboSimSystem</plugin>
+            </xacro:if>
           </xacro:if>
         </hardware>
@@ -58,8 +68,8 @@
       </xacro:unless>
       <!-- wheels -->
-      <xacro:ros2_control_wheel side="front_right" />
-      <xacro:ros2_control_wheel side="front_left" />
-      <xacro:ros2_control_wheel side="rear_right" />
-      <xacro:ros2_control_wheel side="rear_left" />
+      <xacro:ros2_control_wheel side="front_right" sim_type="${sim_type}"/>
+      <xacro:ros2_control_wheel side="front_left" sim_type="${sim_type}"/>
+      <xacro:ros2_control_wheel side="rear_right" sim_type="${sim_type}"/>
+      <xacro:ros2_control_wheel side="rear_left" sim_type="${sim_type}"/>
     </ros2_control>
   </xacro:macro>

File: omni_base_description/urdf/base/base.urdf.xacro (robot description, xacro)
@@ -117,3 +117,45 @@
     <xacro:base_gazebo name="${name}"/>
   </xacro:macro>
+  <xacro:macro name="base_mj" params="mj_control world_name">
+    <xacro:include filename="$(find omni_base_description)/mujoco/mj_tags.xacro" />
+    <xacro:include filename="$(find pal_mujoco_scenes)/scenes/${world_name}.xacro" />
+    <mujoco_inputs>
+      <!-- Mujoco environment -->
+      <scene>
+        <xacro:mj_scene/>
+      </scene>
+      <raw_inputs>
+        <!-- Actuator-->
+          <actuator>
+            <xacro:mj_base_actuators mj_control="${mj_control}"/>
+          </actuator>
+          <default>
+            <default class="visual">
+              <geom group="2" type="mesh" contype="0" conaffinity="0"/>
+            </default>
+            <default class="collision">
+              <geom group="3" type="mesh"/>
+            </default>
+          </default>
+      </raw_inputs>
+      <processed_inputs>
+        <!-- Specifying decompose_mesh will set the `decompose` flag when using obj2mjcf -->
+        <decompose_mesh mesh_name="wheel_link" threshold="0.5"/>
+        <decompose_mesh mesh_name="wheel_link_reflected" threshold="0.5"/>
+        <!-- The camera with the specified values will be added at the specified site name. -->
+        <!-- The position and quaterinion will be filled in by the converter -->
+        <!-- <camera site="{site_name}" name="{camera_name}" fovy="{fovy_value}" mode="{mode_type}" resolution="{resolution values}"/> -->
+        <!-- Adds a lidar tag below a site tag to support a lidar sensor. -->
+        <!-- In the URDF, we assume that that the sensor frame has the Z-axis pointed directly up in the sensor -->
+        <!-- frame. This tag will create rangefinders in the MJCF between min_angle and max_angle at each -->
+        <!-- angle_increment rotated about the replicate frame's Y axis. The hardware intercface then combines -->
+        <!-- them into a single LaserScan message. -->
+        <!-- <lidar ref_site="{link_name}" sensor_name="{sensor_name}" min_angle="{min_angle_value}" max_angle="{max_angle_value}" angle_increment="{angle_increment_value}" /> -->
+        <!-- The element with the type and name as listed below will be modified with the remaining attributes -->
+        <!-- If the attribute already existed, it will be overwritten -->
+        <!-- Note that the type and name elements are required -->
+        <!-- <modify_element type="{element_type}" name="{element_name}" frictionloss="{value}" damping="{value}"/> -->
+      </processed_inputs>
+    </mujoco_inputs>
+  </xacro:macro>
 </robot>

File: omni_base_description/urdf/objects/antenna.urdf.xacro (robot description, xacro)
@@ -16,4 +16,5 @@
   <xacro:macro name="antenna" params="name parent *origin reflect:=1">
     <link name="${name}_link">
+      <xacro:property name="suffix" value="${'_reflected' if reflect == -1 else ''}" />
       <inertial>
         <origin xyz="0.027807 ${reflect * -0.0085125} 0.015138" rpy="0 0 0" />
@@ -25,10 +26,5 @@
         <origin xyz="0 0 0" rpy="0 0 0" />
         <geometry>
-          <xacro:if value="${reflect == 1}">
-            <mesh filename="package://omni_base_description/meshes/base/base_antenna_link.stl" scale="1 1 1" />
-          </xacro:if>
-          <xacro:unless value="${reflect == 1}">
-            <mesh filename="package://omni_base_description/meshes/base/base_antenna_link_mirror.stl" scale="1 1 1"/>
-          </xacro:unless>
+          <mesh filename="package://omni_base_description/meshes/base/base_antenna_link${suffix}.stl"/>
         </geometry>
         <material name="">
@@ -39,10 +35,5 @@
         <origin xyz="0 0 0" rpy="0 0 0" />
         <geometry>
-          <xacro:if value="${reflect == 1}">
-            <mesh filename="package://omni_base_description/meshes/base/base_antenna_link.stl" scale="1 1 1" />
-          </xacro:if>
-          <xacro:unless value="${reflect == 1}">
-            <mesh filename="package://omni_base_description/meshes/base/base_antenna_link_mirror.stl" scale="1 1 1"/>
-          </xacro:unless>
+          <mesh filename="package://omni_base_description/meshes/base/base_antenna_link${suffix}.stl" />
         </geometry>
       </collision>

File: omni_base_description/urdf/wheels/wheel.ros2_control.xacro (robot description, xacro)
@@ -15,5 +15,5 @@
   <!-- TODO Compute real wheel max velocity -->
   <!-- MACRO DEFINITION -->
-  <xacro:macro name="ros2_control_wheel" params="side">
+  <xacro:macro name="ros2_control_wheel" params="side sim_type:=^|gazebo">
     <joint name="wheel_${side}_joint">
       <command_interface name="velocity"/>
@@ -22,5 +22,10 @@
     <transmission name="wheel_${side}_trans">
       <plugin>transmission_interface/SimpleTransmission</plugin>
-      <actuator name="wheel_${side}_actuator" role="actuator1"/>
+      <xacro:if value="${sim_type == 'mujoco-ros2-control'}">
+        <actuator name="wheel_${side}_joint" role="actuator1"/>
+      </xacro:if>
+      <xacro:unless value="${sim_type == 'mujoco-ros2-control'}">
+        <actuator name="wheel_${side}_actuator" role="actuator1"/>
+      </xacro:unless>
       <joint name="wheel_${side}_joint" role="joint1">
         <mechanical_reduction>1.0</mechanical_reduction>

File: omni_base_description/urdf/wheels/wheel.urdf.xacro (robot description, xacro)
@@ -20,4 +20,5 @@
   <xacro:macro name="wheel" params="side parent sagital_reflect frontal_reflect radius width torque velocity sagital_separation frontal_separation">
     <link name="suspension_${side}_link">
+      <xacro:property name="suffix" value="${'_reflected' if sagital_reflect == -1 else ''}" />
       <inertial>
         <origin xyz="-0.058182 ${frontal_reflect * sagital_reflect * -0.0043908} -0.0057695" rpy="0 0 0" />
@@ -30,8 +31,8 @@
         <geometry>
           <xacro:if value="${frontal_reflect == 1}">
-            <mesh filename="package://omni_base_description/meshes/wheels/suspension_front_link.stl" scale="1 1 1"/>
+            <mesh filename="package://omni_base_description/meshes/wheels/suspension_front_link${suffix}.stl"/>
           </xacro:if>
           <xacro:unless value="${frontal_reflect == 1}">
-            <mesh filename="package://omni_base_description/meshes/wheels/suspension_rear_link.stl" scale="1 1 1"/>
+            <mesh filename="package://omni_base_description/meshes/wheels/suspension_rear_link${suffix}.stl"/>
           </xacro:unless>
         </geometry>
@@ -44,8 +45,8 @@
         <geometry>
           <xacro:if value="${frontal_reflect == 1}">
-            <mesh filename="package://omni_base_description/meshes/wheels/suspension_front_link.stl" scale="1 1 1"/>
+            <mesh filename="package://omni_base_description/meshes/wheels/suspension_front_link${suffix}.stl"/>
           </xacro:if>
           <xacro:unless value="${frontal_reflect == 1}">
-            <mesh filename="package://omni_base_description/meshes/wheels/suspension_rear_link.stl" scale="1 1 1"/>
+            <mesh filename="package://omni_base_description/meshes/wheels/suspension_rear_link${suffix}.stl"/>
           </xacro:unless>
         </geometry>
@@ -62,4 +63,5 @@
     </joint>
     <link name="wheel_${side}_link">
+      <xacro:property name="suffix" value="${'_reflected' if sagital_reflect == -1 else ''}" />
       <inertial>
         <origin xyz="${frontal_reflect * 5.4922E-09} ${frontal_reflect * sagital_reflect * 6.9775E-05} ${sagital_reflect * 0.011144}" rpy="0 0 0" />
@@ -71,10 +73,5 @@
         <origin xyz="0 0 0" rpy="0 0 0" />
         <geometry>
-          <xacro:if value="${sagital_reflect == 1}">
-            <mesh filename="package://omni_base_description/meshes/wheels/wheel_link.stl" scale="1 1 1"/>
-          </xacro:if>
-          <xacro:unless value="${sagital_reflect == 1}">
-            <mesh filename="package://omni_base_description/meshes/wheels/wheel_link_reverted.stl" scale="1 1 1"/>
-          </xacro:unless>
+          <mesh filename="package://omni_base_description/meshes/wheels/wheel_link${suffix}.stl"/>
         </geometry>
         <material name="DarkGrey"/>
